File: pcb/direct-digital-synthesis.kicad_pcb (KiCad board)
At the start: 4 copper layers, 100 parts, among them IC1 IS45S16800F-7TLA2, J1 TagConnect_TC2030, U1 STM32H723ZGT6, U2 AD5445YCPZ, U3 REF5010AID, U4 LTC3260EDE-PBF, U5 LMR36015FBRNXR, U6 OPA810IDR

Commit message: Updated pcb and src
Parts:
- added C19: 1u, Capacitor_SMD:C_0603_1608Metric, F.Cu at (299.9, 204.0)
- added C20: 2u2, Capacitor_SMD:C_0603_1608Metric, F.Cu at (301.9, 173.3)
- added C21: 1u, Capacitor_SMD:C_0603_1608Metric, F.Cu at (292.9, 198.0)
- added C22: 1u, Capacitor_SMD:C_0603_1608Metric, F.Cu at (293.6, 195.7)
- added C23: 100n, Capacitor_SMD:C_0603_1608Metric, F.Cu at (312.4, 150.7)
- added C24: 100n, Capacitor_SMD:C_0603_1608Metric, F.Cu at (333.3, 208.8)
- added C25: 100n, Capacitor_SMD:C_0603_1608Metric, F.Cu at (312.1, 217.6)
- added C26: 100n, Capacitor_SMD:C_0603_1608Metric, F.Cu at (269.9, 208.4)
- added C27: 100n, Capacitor_SMD:C_0603_1608Metric, F.Cu at (268.8, 183.7)
- added J2: MEM2061-01-188-00-A, Custom_Connectors:MEM20610118800A, F.Cu at (315.7, 137.6)
- added J3: Barrel_Jack_Switch, Connector_BarrelJack:BarrelJack_Horizontal, F.Cu at (168.7, 108.1)
- added LED1: IN-S66TBTRGB, Custom_LEDs:INS66TBTRGB, F.Cu at (330.2, 209.2)
- added R10: 22R, Resistor_SMD:R_0603_1608Metric, F.Cu at (282.3, 197.8)
- added R11: 22R, Resistor_SMD:R_0603_1608Metric, F.Cu at (282.3, 199.5)
- added R12: 22R, Resistor_SMD:R_0603_1608Metric, F.Cu at (282.3, 201.2)
- added R13: 22R, Resistor_SMD:R_0603_1608Metric, F.Cu at (282.3, 203.9)
- added R14: 22R, Resistor_SMD:R_0603_1608Metric, F.Cu at (282.3, 205.6)
- added R15: 22R, Resistor_SMD:R_0603_1608Metric, F.Cu at (282.3, 207.3)
- added R16: 22R, Resistor_SMD:R_0603_1608Metric, F.Cu at (282.3, 209.0)
- added R17: 10k, Resistor_SMD:R_0603_1608Metric, F.Cu at (309.3, 150.7)
- added R18: 100R, Resistor_SMD:R_0603_1608Metric, F.Cu at (326.9, 209.9)
- added R19: 100R, Resistor_SMD:R_0603_1608Metric, F.Cu at (326.9, 208.3)
- added R20: 100R, Resistor_SMD:R_0603_1608Metric, F.Cu at (330.1, 207.0)
- added R21: 22R, Resistor_SMD:R_0603_1608Metric, F.Cu at (282.4, 212.0)
- added R22: 0R, Resistor_SMD:R_0603_1608Metric, F.Cu at (307.0, 151.5)
- added R23: 22R, Resistor_SMD:R_0603_1608Metric, F.Cu at (311.4, 210.3)
- added R24: 22R, Resistor_SMD:R_0603_1608Metric, F.Cu at (264.9, 206.7)
- added R25: 22R, Resistor_SMD:R_0603_1608Metric, F.Cu at (264.9, 205.1)
- added R26: 22R, Resistor_SMD:R_0603_1608Metric, F.Cu at (264.9, 203.4)
- added R27: 22R, Resistor_SMD:R_0603_1608Metric, F.Cu at (264.9, 201.7)
- added R28: 22R, Resistor_SMD:R_0603_1608Metric, F.Cu at (264.9, 200.0)
- added R30: 22R, Resistor_SMD:R_0603_1608Metric, F.Cu at (264.2, 183.6)
- added R31: 22R, Resistor_SMD:R_0603_1608Metric, F.Cu at (264.2, 181.9)
- added R32: 22R, Resistor_SMD:R_0603_1608Metric, F.Cu at (264.2, 180.1)
- added R33: 22R, Resistor_SMD:R_0603_1608Metric, F.Cu at (264.2, 178.4)
- added R34: 22R, Resistor_SMD:R_0603_1608Metric, F.Cu at (264.2, 176.6)
- added R35: 22R, Resistor_SMD:R_0603_1608Metric, F.Cu at (264.2, 174.9)
- added R36: 22R, Resistor_SMD:R_0603_1608Metric, F.Cu at (264.2, 173.2)
- added R37: 50k, Resistor_SMD:R_0603_1608Metric, F.Cu at (244.9, 187.2)
- added R44: 100k, Resistor_SMD:R_0603_1608Metric, F.Cu at (226.8, 191.9)
- added R45: 100k, Resistor_SMD:R_0603_1608Metric, F.Cu at (226.8, 193.5)
- added R6: 22R, Resistor_SMD:R_0603_1608Metric, F.Cu at (284.5, 175.2)
- added R8: 22R, Resistor_SMD:R_0603_1608Metric, F.Cu at (284.5, 178.6)
- added R9: 22R, Resistor_SMD:R_0603_1608Metric, F.Cu at (282.3, 196.1)
- added TP18: MCU_OSC_IN, TestPoint:TestPoint_THTPad_D1.5mm_Drill0.7mm, F.Cu at (308.4, 209.5)
- added U3: PCHCS541QWRKSRQ1, Custom_LineDrivers:RKS0020B_VQFN_TEX-M, F.Cu at (269.8, 179.6)
- added U8: OPA810IDR, Custom_OpAmps:SOIC8_D_TEX-M, F.Cu at (221.0, 191.1)
- added Y1: ECS-2520MVQ-240-BS-TR, Custom_Oscillators:ECS2520MVQ240BSTR, F.Cu at (312.1, 214.3)
- C10: value 100n -> 1u
- C12: value 1u -> 10u; footprint Capacitor_SMD:C_0603_1608Metric -> Capacitor_SMD:C_0805_2012Metric
- C13: value 2u2 -> 1u
- C15: value 2u2 -> 100n
- C18: value 1u -> 2u2
- C52: renamed from C43; moved to B.Cu
- C53: renamed from C44; moved to B.Cu
- C54: renamed from C45; moved to B.Cu
- C55: renamed from C46; moved to B.Cu
- C56: renamed from C47; moved to B.Cu
- C57: renamed from C48; moved to B.Cu
- C58: renamed from C49; moved to B.Cu
- C59: renamed from C50; moved to B.Cu
- C60: renamed from C51; moved to B.Cu
- IC1: value IS45S16800F-7TLA2 -> IS42S16160J-7TLI; moved to B.Cu
- R5: value 2k2 -> 22R
- U1: value STM32H723ZGT6 -> STM32H750IBT6; footprint Package_QFP:LQFP-144_20x20mm_P0.5mm -> Package_QFP:LQFP-176_24x24mm_P0.5mm
- U2: value AD5445YCPZ -> PCHCS541QWRKSRQ1; footprint Custom_DACs:CP_20_1_ADI-M -> Custom_LineDrivers:RKS0020B_VQFN_TEX-M
- U6: value OPA810IDR -> AD5445YCPZ; footprint Custom_OpAmps:SOIC8_D_TEX-M -> Custom_DACs:CP_20_1_ADI-M
- moved FID7 457.3 mm to (450.7, 242.6)
- moved H1 457.3 mm to (439.5, 238.3)
- moved H2 457.3 mm to (439.5, 248.5)
- moved H3 457.3 mm to (439.5, 258.6)
- moved TP12 457.3 mm to (445.4, 301.1)
- moved TP16 457.3 mm to (449.7, 301.1)
- moved TP4 457.3 mm to (436.7, 301.1)
- moved TP8 457.3 mm to (441.0, 301.1)
- moved FID1 457.3 mm to (451.2, 236.0)
- moved FID2 457.3 mm to (451.2, 239.6)
- moved FID3 457.3 mm to (454.8, 236.0)
- moved FID4 457.3 mm to (454.8, 239.6)
- moved FID5 457.3 mm to (458.3, 236.0)
- moved FID6 457.3 mm to (458.3, 239.6)
- moved H4 457.3 mm to (439.5, 268.8)
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- renumbered C23 to C28, C28 to C29, C24 to C30, C26 to C31, C19 to C32, C22 to C33, C20 to C34, C25 to C35, C32 to C36, C27 to C37, C34 to C38, C29 to C39, C36 to C40, C21 to C41, C35 to C42, C38 to C43, C33 to C44, C40 to C45, C37 to C46, C30 to C47, C31 to C48, C39 to C49, C41 to C50, C42 to C51, R6 to R29, R10 to R38, R11 to R39, R12 to R40, R13 to R41, R8 to R42, R9 to R43, U3 to U5, U5 to U7
Connections:
- C10 pad 1: /MCU_NRST -> +3.3V
- C13 pad 1: Net-(C13-Pad1) -> +3.3V
- C15 pad 1: Net-(C15-Pad1) -> /MCU_NRST
- C18 pad 1: +3.3V -> Net-(C18-Pad1)
- IC1 pad 10: /SDRAM_DQ5 -> /SDRAM.DQ5
- IC1 pad 11: /SDRAM_DQ6 -> /SDRAM.DQ6
- IC1 pad 13: /SDRAM_DQ7 -> /SDRAM.DQ7
- IC1 pad 2: /SDRAM_DQ0 -> /SDRAM.DQ0
- IC1 pad 36: unconnected-(IC1-NC_1-Pad36) -> /SDRAM_A12
- IC1 pad 4: /SDRAM_DQ1 -> /SDRAM.DQ1
- IC1 pad 42: /SDRAM_DQ8 -> /SDRAM.DQ8
- IC1 pad 44: /SDRAM_DQ9 -> /SDRAM.DQ9
- IC1 pad 45: /SDRAM_DQ10 -> /SDRAM.DQ10
- IC1 pad 47: /SDRAM_DQ11 -> /SDRAM.DQ11
- IC1 pad 48: /SDRAM_DQ12 -> /SDRAM.DQ12
- IC1 pad 5: /SDRAM_DQ2 -> /SDRAM.DQ2
- IC1 pad 50: /SDRAM_DQ13 -> /SDRAM.DQ13
- IC1 pad 51: /SDRAM_DQ14 -> /SDRAM.DQ14
- IC1 pad 53: /SDRAM_DQ15 -> /SDRAM.DQ15
- IC1 pad 7: /SDRAM_DQ3 -> /SDRAM.DQ3
- IC1 pad 8: /SDRAM_DQ4 -> /SDRAM.DQ4
- R29 pad 1: unconnected-(R6-Pad1) -> Net-(U3-Y1)
- R29 pad 2: unconnected-(R6-Pad2) -> /DAC.DB7
- R5 pad 1: Net-(D6-K) -> Net-(U1-PI0)
- R5 pad 2: GND -> /MCU_DAC.DB0
- R7 pad 1: unconnected-(R7-Pad1) -> Net-(U1-PI2)
- R7 pad 2: unconnected-(R7-Pad2) -> /MCU_DAC.DB2
- U1 pad 102: unconnected-(U1-PA10-Pad102) -> GND
- U1 pad 103: unconnected-(U1-PA11-Pad103) -> +3.3V
- U1 pad 104: unconnected-(U1-PA12-Pad104) -> /SDRAM.DQ0
- U1 pad 105: /MCU_SWDIO -> /SDRAM.DQ1
- U1 pad 106: Net-(C15-Pad1) -> /SDRAM_A12
- U1 pad 107: GND -> unconnected-(U1-PG3-Pad107)
- U1 pad 108: +3.3V -> /SDRAM_BA0
- U1 pad 109: /MCU_SWCLK -> /SDRAM_BA1
- U1 pad 11: unconnected-(U1-PF1-Pad11) -> Net-(U1-PI9)
- U1 pad 112: unconnected-(U1-PC11-Pad112) -> /SDRAM_CLK
- U1 pad 113: unconnected-(U1-PC12-Pad113) -> GND
- U1 pad 114: unconnected-(U1-PD0-Pad114) -> +3.3V
- U1 pad 117: unconnected-(U1-PD3-Pad117) -> /SD_DAT0
- U1 pad 118: unconnected-(U1-PD4-Pad118) -> /SD_DAT1
- U1 pad 12: unconnected-(U1-PF2-Pad12) -> Net-(U1-PI10)
- U1 pad 120: GND -> unconnected-(U1-PA9-Pad120)
- U1 pad 121: +3.3V -> unconnected-(U1-PA10-Pad121)
- U1 pad 124: unconnected-(U1-PG9-Pad124) -> /MCU_SWDIO
- U1 pad 125: unconnected-(U1-PG10-Pad125) -> Net-(C20-Pad1)
- U1 pad 126: unconnected-(U1-PG11-Pad126) -> GND
- U1 pad 127: unconnected-(U1-PG12-Pad127) -> +3.3V
- U1 pad 13: unconnected-(U1-PF3-Pad13) -> Net-(U1-PI11)
- U1 pad 130: GND -> unconnected-(U1-PH15-Pad130)
- U1 pad 131: +3.3V -> Net-(U1-PI0)
- U1 pad 132: unconnected-(U1-PG15-Pad132) -> Net-(U1-PI1)
- U1 pad 133: /MCU_SWO -> Net-(U1-PI2)
- U1 pad 134: unconnected-(U1-PB4(NJTRST)-Pad134) -> Net-(U1-PI3)
- U1 pad 135: unconnected-(U1-PB5-Pad135) -> GND
- U1 pad 136: unconnected-(U1-PB6-Pad136) -> +3.3V
- U1 pad 137: unconnected-(U1-PB7-Pad137) -> /MCU_SWCLK
- U1 pad 138: GND -> unconnected-(U1-PA15-Pad138)
- U1 pad 139: unconnected-(U1-PB8-Pad139) -> /SD_DAT2
- U1 pad 14: unconnected-(U1-PF4-Pad14) -> GND
- U1 pad 140: unconnected-(U1-PB9-Pad140) -> /SD_DAT3
- U1 pad 141: unconnected-(U1-PE0-Pad141) -> Net-(U1-PC12)
- U1 pad 142: unconnected-(U1-PE1-Pad142) -> /SDRAM.DQ2
- U1 pad 143: +3.3V -> /SDRAM.DQ3
- U1 pad 144: +3.3V -> /SD_CMD
- U1 pad 15: unconnected-(U1-PF5-Pad15) -> +3.3V
- U1 pad 16: GND -> /SDRAM_A0
- U1 pad 17: +3.3V -> /SDRAM_A1
- U1 pad 18: unconnected-(U1-PF6-Pad18) -> /SDRAM_A2
- U1 pad 19: unconnected-(U1-PF7-Pad19) -> /SDRAM_A3
- U1 pad 20: unconnected-(U1-PF8-Pad20) -> /SDRAM_A4
- U1 pad 21: unconnected-(U1-PF9-Pad21) -> /SDRAM_A5
- U1 pad 22: unconnected-(U1-PF10-Pad22) -> GND
- U1 pad 23: unconnected-(U1-PH0-Pad23) -> +3.3V
- U1 pad 25: /MCU_NRST -> unconnected-(U1-PF7-Pad25)
- U1 pad 29: unconnected-(U1-PC3_C-Pad29) -> /MCU_OSC_IN
- U1 pad 30: +3.3V -> unconnected-(U1-PH1-Pad30)
- U1 pad 31: GND -> /MCU_NRST
- U1 pad 32: +3.3V -> /SDRAM_NWE
- U1 pad 33: +3.3V -> unconnected-(U1-PC1-Pad33)
- U1 pad 34: unconnected-(U1-PA0-Pad34) -> /SDRAM_NCS
- U1 pad 35: unconnected-(U1-PA1-Pad35) -> /SDRAM_CKE
- U1 pad 36: unconnected-(U1-PA2-Pad36) -> +3.3V
- U1 pad 37: unconnected-(U1-PA3-Pad37) -> GND
- U1 pad 38: GND -> +3.3V
- U1 pad 41: unconnected-(U1-PA5-Pad41) -> Net-(U1-PA1)
- U1 pad 43: unconnected-(U1-PA7-Pad43) -> /MCU_LED_R
- U1 pad 44: unconnected-(U1-PC4-Pad44) -> /MCU_LED_G
- U1 pad 45: unconnected-(U1-PC5-Pad45) -> /MCU_LED_B
- U1 pad 48: unconnected-(U1-PB2-Pad48) -> GND
- U1 pad 49: unconnected-(U1-PF11-Pad49) -> +3.3V
- U1 pad 51: GND -> unconnected-(U1-PA5-Pad51)
- U1 pad 52: +3.3V -> unconnected-(U1-PA6-Pad52)
- U1 pad 59: unconnected-(U1-PE8-Pad59) -> /SDRAM_NRAS
- U1 pad 60: unconnected-(U1-PE9-Pad60) -> /SDRAM_A6
- U1 pad 63: unconnected-(U1-PE10-Pad63) -> /SDRAM_A7
- U1 pad 64: unconnected-(U1-PE11-Pad64) -> /SDRAM_A8
- U1 pad 65: unconnected-(U1-PE12-Pad65) -> /SDRAM_A9
- U1 pad 66: unconnected-(U1-PE13-Pad66) -> /SDRAM_A10
- U1 pad 67: unconnected-(U1-PE14-Pad67) -> /SDRAM_A11
- U1 pad 68: unconnected-(U1-PE15-Pad68) -> /SDRAM.DQ4
- U1 pad 69: unconnected-(U1-PB10-Pad69) -> /SDRAM.DQ5
- U1 pad 7: unconnected-(U1-PC13-Pad7) -> Net-(U1-PI8)
- U1 pad 70: unconnected-(U1-PB11-Pad70) -> /SDRAM.DQ6
- U1 pad 71: Net-(C13-Pad1) -> GND
- U1 pad 73: unconnected-(U1-PB12-Pad73) -> /SDRAM.DQ7
- U1 pad 74: unconnected-(U1-PB13-Pad74) -> /SDRAM.DQ8
- U1 pad 75: unconnected-(U1-PB14-Pad75) -> /SDRAM.DQ9
- U1 pad 76: unconnected-(U1-PB15-Pad76) -> /SDRAM.DQ10
- U1 pad 77: unconnected-(U1-PD8-Pad77) -> /SDRAM.DQ11
- U1 pad 78: unconnected-(U1-PD9-Pad78) -> /SDRAM.DQ12
- U1 pad 81: unconnected-(U1-PD12-Pad81) -> Net-(C18-Pad1)
- U1 pad 82: unconnected-(U1-PD13-Pad82) -> +3.3V
- U1 pad 83: GND -> unconnected-(U1-PH6-Pad83)
- U1 pad 84: +3.3V -> unconnected-(U1-PH7-Pad84)
- U1 pad 90: unconnected-(U1-PG5-Pad90) -> GND
- U1 pad 91: unconnected-(U1-PG6-Pad91) -> +3.3V
- U1 pad 94: GND -> unconnected-(U1-PB14-Pad94)
- U1 pad 95: +3.3V -> unconnected-(U1-PB15-Pad95)
- U1 pad 96: unconnected-(U1-PC6-Pad96) -> /SDRAM.DQ13
- U1 pad 97: unconnected-(U1-PC7-Pad97) -> /SDRAM.DQ14
- U1 pad 98: unconnected-(U1-PC8-Pad98) -> /SDRAM.DQ15
- U2 pad 10: /DAC_DB3 -> GND
- U2 pad 11: /DAC_DB2 -> Net-(U2-Y8)
- U2 pad 12: /DAC_DB1 -> Net-(U2-Y7)
- U2 pad 13: /DAC_DB0 -> Net-(U2-Y6)
- U2 pad 14: /DAC_NCS -> Net-(U2-Y5)
- U2 pad 15: /DAC_NRW -> unconnected-(U2-Y4-Pad15)
- U2 pad 16: +3.3V -> unconnected-(U2-Y3-Pad16)
- U2 pad 17: /VREF_+10V -> unconnected-(U2-Y2-Pad17)
- U2 pad 18: /DAC_RFB -> Net-(U2-Y1)
- U2 pad 19: /DAC_IOUT1 -> GND
- U2 pad 2: /DAC_DB11 -> /MCU_DAC_NCS
- U2 pad 20: GND -> +3.3V
- U2 pad 3: /DAC_DB10 -> GND
- U2 pad 4: /DAC_DB9 -> GND
- U2 pad 5: /DAC_DB8 -> GND
- U2 pad 6: /DAC_DB7 -> /MCU_DAC.DB11
- U2 pad 7: /DAC_DB6 -> /MCU_DAC.DB10
- U2 pad 8: /DAC_DB5 -> /MCU_DAC.DB9
- U2 pad 9: /DAC_DB4 -> /MCU_DAC.DB8
- U6 pad 1: unconnected-(U6-NC-Pad1) -> GND
- U6 pad 2: unconnected-(U6-VIN--Pad2) -> /DAC.DB11
- U6 pad 3: unconnected-(U6-VIN+-Pad3) -> /DAC.DB10
- U6 pad 4: -12V -> /DAC.DB9
- U6 pad 5: unconnected-(U6-NC-Pad5) -> /DAC.DB8
- U6 pad 6: unconnected-(U6-VO-Pad6) -> /DAC.DB7
- U6 pad 7: +12V -> /DAC.DB6
- U6 pad 8: unconnected-(U6-NC-Pad8) -> /DAC.DB5
Other:
- board outline added: 341 x 224.6 mm

Commit message: pcb update
Parts:
- removed the C47 at (226.1, 189.6)
- removed the C48 at (216.0, 192.5)
- removed the R17 at (309.3, 150.7)
- removed the R44 at (226.8, 191.9)
- added C2: 100n, Capacitor_SMD:C_0603_1608Metric, F.Cu at (419.8, 119.6)
- added C49: 100n, Capacitor_SMD:C_0603_1608Metric, F.Cu at (227.5, 194.2)
- added C50: 100n, Capacitor_SMD:C_0603_1608Metric, F.Cu at (230.1, 188.1)
- added R1: 10k, Resistor_SMD:R_0603_1608Metric, F.Cu at (419.8, 122.1)
- added R18: 50k, Resistor_SMD:R_0603_1608Metric, F.Cu at (419.8, 124.6)
- added R46: 10k, Resistor_SMD:R_0603_1608Metric, F.Cu at (229.9, 193.4)
- added R47: 20k, Resistor_SMD:R_0603_1608Metric, F.Cu at (229.9, 195.0)
- added R48: 20k, Resistor_SMD:R_0603_1608Metric, F.Cu at (226.1, 190.9)
- R45: value 100k -> 20k
- U8: value OPA810IDR -> OPA2810IDGKR; footprint Custom_OpAmps:SOIC8_D_TEX-M -> Custom_OpAmps:DGK0008A_N
- moved TP1 48.5 mm to (322.8, 223.8)
- moved U8 9.13 mm to (230.1, 190.8), turned to 180 degrees
- moved R45 8.31 mm to (234.9, 191.8)
- moved C13 3.61 mm to (298.1, 138.8)
- moved R23 3.61 mm to (304.6, 154.2)
- moved C24 3.61 mm to (310.0, 153.4)
- moved J2 3.61 mm to (313.3, 140.3)
- renumbered C9 to C10, C10 to C11, C11 to C12, C12 to C13, C13 to C14, C14 to C15, C15 to C16, C16 to C17, C17 to C18, C18 to C19, C19 to C20, C20 to C21, C21 to C22, C22 to C23, C23 to C24, C24 to C25, C25 to C26, C26 to C27, C27 to C28, C28 to C29, C2 to C3, C29 to C30, C30 to C31, C31 to C32, C32 to C34, C34 to C36, C36 to C37, C37 to C38, C38 to C39, C3 to C4, C39 to C40, C40 to C41, C41 to C42, C42 to C43, C43 to C44, C44 to C45, C45 to C46, C46 to C47, C49 to C48, C4 to C5, C50 to C51, C51 to C52, C52 to C53, C53 to C54, C54 to C55, C55 to C56, C56 to C57, C57 to C58, C58 to C59, C5 to C6, C59 to C60, C60 to C61, C6 to C7, C7 to C8, C8 to C9, R9 to R10, R10 to R11, R11 to R12, R12 to R13, R13 to R14, R14 to R15, R15 to R16, R16 to R17, R18 to R19, R1 to R2, R19 to R20, R20 to R21, R21 to R22, R22 to R23, R23 to R24, R24 to R25, R25 to R26, R26 to R27, R27 to R28, R28 to R29, R2 to R3, R29 to R30, R30 to R31, R31 to R32, R32 to R33, R33 to R34, R34 to R35, R35 to R36, R36 to R37, R37 to R38, R38 to R39, R3 to R4, R39 to R40, R40 to R41, R41 to R42, R42 to R43, R43 to R44, R4 to R5, R5 to R6, R6 to R7, R7 to R8, R8 to R9
Connections:
- net /SD_NCD renamed /SD_CD
- R45 pad 2: GND -> Net-(R45-Pad2)
- U8 pad 1: unconnected-(U8-NC-Pad1) -> Net-(R45-Pad2)
- U8 pad 5: unconnected-(U8-NC-Pad5) -> GND
- U8 pad 6: /OPAMP_VOUT -> Net-(U8B-IN-)
- U8 pad 7: +12V -> /OPAMP_VOUT
- U8 pad 8: unconnected-(U8-NC-Pad8) -> +12V

Commit message: pcb update
Parts:
- added Q1: PMPB27EPZ, Custom_MOSFETs:DFN-2020MD-6, F.Cu at (168.8, 114.0)
- moved R1 255.1 mm to (164.8, 112.6), turned to -90 degrees
- moved C2 253.5 mm to (166.4, 112.6), turned to -90 degrees
- moved R18 116.0 mm to (307.6, 154.2), turned to -90 degrees

Commit message: update pcb
Parts:
- removed the C43 at (239.4, 120.6)
- removed the R46 at (229.9, 193.4)
- removed the R47 at (229.9, 195.0)
- removed the R48 at (226.1, 190.9)
- removed the U2 at (270.9, 204.2)
- removed the U7 at (147.2, 122.6)
- removed the U8 at (230.1, 190.8)
- added C1: 100n, Capacitor_SMD:C_0603_1608Metric, F.Cu at (356.3, 260.8)
- added C20: 100n, Capacitor_SMD:C_0603_1608Metric, F.Cu at (345.3, 151.6)
- added C25: 100n, Capacitor_SMD:C_0603_1608Metric, F.Cu at (396.9, 144.8)
- added C28: 100n, Capacitor_SMD:C_0603_1608Metric, F.Cu at (398.0, 158.8)
- added C29: 100n, Capacitor_SMD:C_0603_1608Metric, F.Cu at (372.3, 148.4)
- added C30: 100n, Capacitor_SMD:C_0603_1608Metric, F.Cu at (372.5, 141.5)
- added C49: 10u, Capacitor_SMD:C_0805_2012Metric, F.Cu at (239.7, 121.7)
- added C57: 4p7, Capacitor_SMD:C_0603_1608Metric, F.Cu at (220.0, 194.0)
- added C58: 10u, Capacitor_SMD:C_0805_2012Metric, F.Cu at (213.1, 185.8)
- added C59: 10u, Capacitor_SMD:C_0805_2012Metric, F.Cu at (213.1, 188.9)
- added C66: 430p, Capacitor_SMD:C_0603_1608Metric, F.Cu at (178.1, 184.2)
- added C67: 430p, Capacitor_SMD:C_0603_1608Metric, F.Cu at (178.1, 186.7)
- added C68: 10u, Capacitor_SMD:C_0805_2012Metric, F.Cu at (187.8, 194.4)
- added C69: 10u, Capacitor_SMD:C_0805_2012Metric, F.Cu at (187.8, 197.5)
- added C71: 100n, Capacitor_SMD:C_0603_1608Metric, F.Cu at (178.1, 189.2)
- added C72: 100n, Capacitor_SMD:C_0603_1608Metric, F.Cu at (178.1, 191.7)
- added C77: 120p, Capacitor_SMD:C_0603_1608Metric, F.Cu at (182.1, 184.2)
- added C78: 1n8, Capacitor_SMD:C_0603_1608Metric, F.Cu at (182.1, 186.7)
- added C79: 100n, Capacitor_SMD:C_0603_1608Metric, F.Cu at (230.3, 206.8)
- added C80: 100n, Capacitor_SMD:C_0603_1608Metric, F.Cu at (239.9, 209.2)
- added C81: 100n, Capacitor_SMD:C_0603_1608Metric, F.Cu at (238.7, 204.5)
- added J2: Conn_01x07_Socket, Connector_PinSocket_2.54mm:PinSocket_1x07_P2.54mm_Vertical, F.Cu at (353.4, 262.0)
- added L1: 6u8, Custom_Inductors:ASPIAIG-F6060, F.Cu at (142.4, 111.3)
- added R18: 10k, Resistor_SMD:R_0603_1608Metric, F.Cu at (346.1, 149.3)
- added R19: 50k, Resistor_SMD:R_0603_1608Metric, F.Cu at (347.7, 149.3)
- added R21: 10k, Resistor_SMD:R_0603_1608Metric, F.Cu at (368.5, 148.5)
- added R22: 10k, Resistor_SMD:R_0603_1608Metric, F.Cu at (368.5, 143.5)
- added R24: 10k, Resistor_SMD:R_0603_1608Metric, F.Cu at (372.5, 143.1)
- added R26: 22R, Resistor_SMD:R_0603_1608Metric, F.Cu at (348.1, 254.3)
- added R27: 22R, Resistor_SMD:R_0603_1608Metric, F.Cu at (298.1, 150.8)
- added R53: 10k, Resistor_SMD:R_0603_1608Metric, F.Cu at (208.9, 190.6)
- added R54: 20k, Resistor_SMD:R_0603_1608Metric, F.Cu at (208.9, 193.1)
- added R55: 75R, Resistor_SMD:R_0603_1608Metric, F.Cu at (182.1, 189.2)
- added R56: 365R, Resistor_SMD:R_0603_1608Metric, F.Cu at (182.1, 191.7)
- added R57: 442R, Resistor_SMD:R_0603_1608Metric, F.Cu at (186.1, 184.2)
- added R58: 887R, Resistor_SMD:R_0603_1608Metric, F.Cu at (186.1, 186.7)
- added R59: 84R5, Resistor_SMD:R_0603_1608Metric, F.Cu at (186.1, 189.2)
- added R60: 158R, Resistor_SMD:R_0603_1608Metric, F.Cu at (186.1, 191.7)
- added SW1: SW_Push, Button_Switch_THT:SW_PUSH_6mm, F.Cu at (396.9, 137.0)
- added SW2: SW_Push, Button_Switch_THT:SW_PUSH_6mm, F.Cu at (398.0, 151.0)
- added TP19: POWER_+15V, TestPoint:TestPoint_Keystone_5000-5004_Miniature, F.Cu at (156.9, 179.8)
- added TP20: POWER_+10V, TestPoint:TestPoint_Keystone_5000-5004_Miniature, F.Cu at (156.9, 184.2)
- added TP21: POWER_-12V, TestPoint:TestPoint_Keystone_5000-5004_Miniature, F.Cu at (156.9, 188.5)
- added TP22: POWER_+12V, TestPoint:TestPoint_Keystone_5000-5004_Miniature, F.Cu at (156.9, 192.8)
- added TP23: POWER_+3V3, TestPoint:TestPoint_Keystone_5000-5004_Miniature, F.Cu at (156.9, 197.2)
- added U1: PEC12R-3225F-S0024, Custom_Encoders:PEC12R3225FS0024, F.Cu at (350.5, 148.5)
- added U10: AD8066ARZ-R7, Custom_OpAmps:R_8_ADI-M, F.Cu at (180.8, 196.7)
- added U11: MCP45HV51-ST, Package_SO:TSSOP-14_4.4x5mm_P0.65mm, F.Cu at (235.1, 208.1)
- added U4: PCHCS541QWRKSRQ1, Custom_LineDrivers:RKS0020B_VQFN_TEX-M, F.Cu at (269.1, 178.8)
- added U6: LMR36015FBRNXR, Custom_PowerModules:RNX0012B, F.Cu at (147.2, 122.6)
- added U9: AD8066ARZ-R7, Custom_OpAmps:R_8_ADI-M, F.Cu at (221.3, 188.9)
- R23: value 0R -> 10k
- R45: renamed from R38; value 50k -> 0R
- R52: renamed from R45; value 20k -> 0R
- TP1, TP18: footprint TestPoint:TestPoint_THTPad_D1.5mm_Drill0.7mm -> TestPoint:TestPoint_Keystone_5000-5004_Miniature
- moved R23 67.9 mm to (372.3, 150.0), turned to 180 degrees
- moved R52 26.3 mm to (208.9, 188.1)
- moved U3 24.5 mm to (269.9, 204.0)
- moved C61 21.4 mm to (208.9, 185.6)
- moved C60 15.5 mm to (212.1, 192.4)
- moved C45 9.17 mm to (202.6, 119.5)
- moved C47 9.17 mm to (202.3, 124.2)
- moved C52 9.17 mm to (207.4, 123.0)
- moved R49 9.17 mm to (203.9, 125.8)
- moved C38 9.17 mm to (198.8, 118.1)
- moved C48 9.17 mm to (198.1, 125.1)
- moved R48 9.17 mm to (205.5, 124.1)
- moved R50 9.17 mm to (194.1, 123.8)
- moved U5 9.17 mm to (198.9, 121.6)
- moved R51 9.17 mm to (195.7, 125.5)
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- renumbered C9 to C10, C24 to C11, C10 to C12, C11 to C13, C12 to C14, C14 to C15, C15 to C16, C26 to C17, C16 to C18, C17 to C19, C13 to C2, C18 to C21, C19 to C22, C20 to C23, C21 to C24, C22 to C26, C23 to C27, C1 to C3, C25 to C31, C27 to C32, C28 to C33, C33 to C34, C29 to C35, C35 to C36, C38 to C37, C30 to C38, C40 to C39, C3 to C4, C31 to C40, C32 to C41, C2 to C42, C34 to C43, C36 to C44, C37 to C45, C45 to C46, C39 to C47, C41 to C48, C4 to C5, C42 to C50, C47 to C51, C44 to C52, C48 to C53, C46 to C54, C51 to C55, C52 to C56, C5 to C6, C49 to C60, C50 to C61, C53 to C62, C54 to C63, C55 to C64, C56 to C65, C6 to C7, C57 to C70, C58 to C73, C59 to C74, C60 to C75, C61 to C76, C7 to C8, C8 to C9, J2 to J1, J1 to J3, J3 to J4, R18 to R1, R24 to R20, R22 to R25, R19 to R28, R20 to R29, R21 to R30, R25 to R31, R26 to R32, R27 to R33, R28 to R34, R29 to R35, R30 to R36, R31 to R37, R32 to R38, R33 to R39, R34 to R40, R35 to R41, R36 to R42, R37 to R43, R1 to R44, R43 to R46, R44 to R47, R39 to R48, R40 to R49, R41 to R50, R42 to R51, U1 to U2, U4 to U5, U5 to U7, U6 to U8
Connections:
- net /POWER_SWITCH renamed /PMOS_DRAIN
- C34 pad 1: +15V -> /POWER_SWITCH_+15V
- C35 pad 1: +15V -> /POWER_SWITCH_+15V
- C36 pad 2: +15V -> /POWER_SWITCH_+15V
- C37 pad 2: +15V -> /POWER_SWITCH_+15V
- C40 pad 1: +15V -> /POWER_SWITCH_+15V
- C51 pad 2: +3.3V -> Net-(JP5-A)
- C52 pad 1: -12V -> Net-(JP3-A)
- C53 pad 1: +3.3V -> Net-(JP5-A)
- C54 pad 1: +12V -> Net-(JP4-A)
- C55 pad 1: +3.3V -> Net-(JP5-A)
- C56 pad 2: +3.3V -> Net-(JP5-A)
- R23 pad 1: Net-(U1-PC12) -> Net-(R21-Pad1)
- R23 pad 2: /SD_CLK -> /UI_ENC_A
- R31 pad 1: Net-(U2-Y1) -> Net-(U3-Y1)
- R32 pad 1: Net-(U2-Y5) -> Net-(U3-Y5)
- R33 pad 1: Net-(U2-Y6) -> Net-(U3-Y6)
- R34 pad 1: Net-(U2-Y7) -> Net-(U3-Y7)
- R35 pad 1: Net-(U2-Y8) -> Net-(U3-Y8)
- R36 pad 1: Net-(U3-Y1) -> Net-(U4-Y1)
- R37 pad 1: Net-(U3-Y2) -> Net-(U4-Y2)
- R38 pad 1: Net-(U3-Y3) -> Net-(U4-Y3)
- R39 pad 1: Net-(U3-Y4) -> Net-(U4-Y4)
- R40 pad 1: Net-(U3-Y5) -> Net-(U4-Y5)
- R41 pad 1: Net-(U3-Y6) -> Net-(U4-Y6)
- R42 pad 1: Net-(U3-Y7) -> Net-(U4-Y7)
- R43 pad 1: Net-(U3-Y8) -> Net-(U4-Y8)
- R46 pad 1: +3.3V -> Net-(JP5-A)
- R48 pad 1: -12V -> Net-(JP3-A)
- R50 pad 1: +12V -> Net-(JP4-A)
- U2 pad 141: Net-(U1-PC12) -> Net-(U2-PC12)
- U2 pad 50: unconnected-(U1-PA4-Pad50) -> /DISP_CS
- U2 pad 51: unconnected-(U1-PA5-Pad51) -> Net-(U2-PA5)
- U2 pad 52: unconnected-(U1-PA6-Pad52) -> /DISP_DC
- U2 pad 53: unconnected-(U1-PA7-Pad53) -> /DISP_DIN
- U2 pad 54: unconnected-(U1-PC4-Pad54) -> /DISP_NRST
- U2 pad 84: unconnected-(U1-PH7-Pad84) -> /UI_SW_A
- U2 pad 85: unconnected-(U1-PH8-Pad85) -> /UI_SW_B
- U2 pad 87: unconnected-(U1-PH10-Pad87) -> /UI_ENC_A
- U2 pad 88: unconnected-(U1-PH11-Pad88) -> /UI_ENC_B
- U2 pad 89: unconnected-(U1-PH12-Pad89) -> /UI_ENC_SW
- U3 pad 15: Net-(U3-Y4) -> unconnected-(U3-Y4-Pad15)
- U3 pad 16: Net-(U3-Y3) -> unconnected-(U3-Y3-Pad16)
- U3 pad 17: Net-(U3-Y2) -> unconnected-(U3-Y2-Pad17)
- U3 pad 2: /MCU_DAC.DB7 -> /MCU_DAC_NCS
- U3 pad 3: /MCU_DAC.DB6 -> GND
- U3 pad 4: /MCU_DAC.DB5 -> GND
- U3 pad 5: /MCU_DAC.DB4 -> GND
- U3 pad 6: /MCU_DAC.DB3 -> /MCU_DAC.DB11
- U3 pad 7: /MCU_DAC.DB2 -> /MCU_DAC.DB10
- U3 pad 8: /MCU_DAC.DB1 -> /MCU_DAC.DB9
- U3 pad 9: /MCU_DAC.DB0 -> /MCU_DAC.DB8
- U5 pad 1: +15V -> /POWER_SWITCH_+15V
- U5 pad 10: +12V -> Net-(JP4-A)
- U5 pad 11: +15V -> /POWER_SWITCH_+15V
- U5 pad 5: -12V -> Net-(JP3-A)
- U5 pad 9: +15V -> /POWER_SWITCH_+15V
- U7 pad 2: +15V -> /POWER_SWITCH_+15V
- U7 pad 6: /VREF_+10V -> Net-(JP2-A)
Routing:
- added copper zone on F.Cu, net /PMOS_DRAIN

Commit message: pcb update
Parts:
- removed the C46 at (144.5, 124.2)
- removed the C57 at (220.0, 194.0)
- removed the C66 at (178.1, 184.2)
- removed the C67 at (178.1, 186.7)
- removed the R25 at (282.4, 212.0)
- removed the R45 at (244.9, 187.2)
- removed the R52 at (208.9, 188.1)
- removed the R53 at (208.9, 190.6)
- removed the R54 at (208.9, 193.1)
- removed the R55 at (182.1, 189.2)
- removed the R56 at (182.1, 191.7)
- removed the R57 at (186.1, 184.2)
- removed R58: 887R, Resistor_SMD:R_0603_1608Metric
- removed the TP18 at (308.4, 209.5)
- removed the U10 at (180.8, 196.7)
- added C39: 100n, Capacitor_SMD:C_0603_1608Metric, F.Cu at (358.4, 198.8)
- added C47: 4p7, Capacitor_SMD:C_0603_1608Metric, F.Cu at (255.7, 222.2)
- added C71: 220p, Capacitor_SMD:C_0603_1608Metric, F.Cu at (253.0, 265.4)
- added C72: 470p, Capacitor_SMD:C_0603_1608Metric, F.Cu at (254.7, 261.2)
- added C82: 100n, Capacitor_SMD:C_0603_1608Metric, F.Cu at (259.9, 205.6)
- added D1: VCAN16A2-03GHE3-08, Custom_TVS:SOT65P230X110-3N, F.Cu at (372.3, 206.8)
- added JP1: ME-100, Custom_Jumpers:ME-100, F.Cu at (365.6, 205.7)
- added JP2: ME-100, Custom_Jumpers:ME-100, F.Cu at (342.8, 174.0)
- added JP3: ME-100, Custom_Jumpers:ME-100, F.Cu at (356.8, 178.7)
- added JP4: ME-100, Custom_Jumpers:ME-100, F.Cu at (357.0, 157.5)
- added JP5: ME-100, Custom_Jumpers:ME-100, F.Cu at (342.3, 197.7)
- added R18: 22R, Resistor_SMD:R_0603_1608Metric, F.Cu at (305.5, 208.1)
- added R41: 20k, Resistor_SMD:R_0603_1608Metric, F.Cu at (258.0, 211.3)
- added R42: 10k, Resistor_SMD:R_0603_1608Metric, F.Cu at (253.4, 217.6)
- added R43: 20k, Resistor_SMD:R_0603_1608Metric, F.Cu at (256.4, 211.3)
- added R50: 59R, Resistor_SMD:R_0603_1608Metric, F.Cu at (249.0, 266.1)
- added R51: 40R2, Resistor_SMD:R_0603_1608Metric, F.Cu at (250.9, 268.3)
- added S1: L102021ML04Q, Custom_Switches:L102021ML04Q, F.Cu at (384.2, 175.0)
- added U12: TLV07IDR, Custom_OpAmps:DGK0008A_N, F.Cu at (258.3, 201.6)
- added U8: AD8066ARZ-R7, Custom_OpAmps:R_8_ADI-M, F.Cu at (257.3, 217.2)
- C59: renamed from C77; value 120p -> 220p
- C60: renamed from C78; value 1n8 -> 470p
- R44: renamed from R59; value 84R5 -> 59R
- R45: renamed from R60; value 158R -> 40R2
- moved TP11 256.9 mm to (239.5, 147.4)
- moved TP3 256.9 mm to (230.8, 147.4)
- moved TP10 256.9 mm to (239.5, 143.1)
- moved TP14 256.9 mm to (243.9, 143.1)
- moved TP15 256.9 mm to (243.9, 147.4)
- moved TP2 256.9 mm to (230.8, 143.1)
- moved TP6 256.9 mm to (235.2, 143.1)
- moved TP7 256.9 mm to (235.2, 147.4)
- moved TP1 256.9 mm to (230.8, 138.7)
- moved TP12 256.9 mm to (239.5, 151.8)
- moved TP13 256.9 mm to (243.9, 138.7)
- moved TP16 256.9 mm to (243.9, 151.8)
- moved TP4 256.9 mm to (230.8, 151.8)
- moved TP5 256.9 mm to (235.2, 138.7)
- moved TP8 256.9 mm to (235.2, 151.8)
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- renumbered C3 to C1, C12 to C10, C13 to C11, C14 to C12, C15 to C13, C16 to C14, C18 to C15, C19 to C16, C21 to C17, C22 to C18, C23 to C19, C4 to C2, C24 to C20, C26 to C21, C27 to C22, C32 to C23, C33 to C24, C34 to C25, C35 to C26, C43 to C27, C36 to C28, C44 to C29, C5 to C3, C38 to C30, C37 to C31, C40 to C32, C39 to C33, C41 to C34, C42 to C35, C50 to C36, C45 to C37, C47 to C38, C6 to C4, C48 to C40, C49 to C41, C52 to C42, C51 to C43, C58 to C44, C59 to C45, C54 to C46, C60 to C48, C61 to C49, C7 to C5, C53 to C50, C55 to C51, C56 to C52, C31 to C53, C62 to C54, C2 to C55, C63 to C56, C64 to C57, C65 to C58, C17 to C6, C70 to C61, C73 to C62, C11 to C63, C68 to C64, C69 to C65, C74 to C66, C71 to C67, C72 to C68, C75 to C69, C8 to C7, C76 to C70, C1 to C73, C20 to C74, C25 to C75, C79 to C76, C80 to C77, C81 to C78, C28 to C79, C9 to C8, C29 to C80, C30 to C81, C10 to C9, J3 to J1, J4 to J2, J1 to J3, J2 to J5, R2 to R1, R26 to R19, R3 to R2, R27 to R20, R31 to R21, R32 to R22, R33 to R23, R34 to R24, R35 to R25, R36 to R26, R37 to R27, R38 to R28, R39 to R29, R4 to R3, R40 to R30, R41 to R31, R42 to R32, R43 to R33, R44 to R34, R46 to R35, R47 to R36, R48 to R37, R49 to R38, R50 to R39, R5 to R4, R51 to R40, R28 to R46, R29 to R47, R30 to R48, R1 to R49, R20 to R5, R18 to R52, R19 to R53, R21 to R54, R22 to R55, R23 to R56, R24 to R57, TP2 to TP1, TP11 to TP10, TP12 to TP11, TP13 to TP12, TP14 to TP13, TP15 to TP14, TP16 to TP15, TP17 to TP16, TP1 to TP17, TP19 to TP18, TP20 to TP19, TP3 to TP2, TP21 to TP20, TP22 to TP21, TP23 to TP22, TP4 to TP3, TP5 to TP4, TP6 to TP5, TP7 to TP6, TP8 to TP7, TP9 to TP8, TP10 to TP9, U2 to U1, U1 to U10, U3 to U2, U4 to U3, U8 to U4, U7 to U6, U6 to U7
Connections:
- net /OPAMP_DC_BIAS_VOUT renamed /OPAMP_FILT_VOUT
- net Net-(JP3-A) renamed /CHGPMP_-LDO
- net Net-(JP4-A) renamed /CHGPMP_+LDO
- net Net-(JP5-A) renamed /SMPS_VOUT
- net Net-(U5-BYP+) renamed /CHGPMP_+BYP
- net Net-(U5-BYP-) renamed /CHGPMP_-BYP
- net Net-(U5-C+) renamed /CHGPMP_+C
- net Net-(U5-C-) renamed /CHGPMP_-C
- net Net-(U5-VOUT) renamed /CHGPMP_VOUT
- net Net-(U6-FB) renamed /SMPS_FB
- net Net-(U6-NC) renamed /SMPS_SW
- net Net-(U6-VCC) renamed /SMPS_VCC
- C36 pad 1: /VREF_+10V -> /OPAMP_VREF
- C59 pad 1: Net-(U10B-IN+) -> Net-(U9A-IN+)
- C60 pad 2: /OPAMP_VOUT_FILT -> Net-(U9A-IN-)
- J5 pad 3: /DISP_DIN -> /DISP_CS
- J5 pad 5: /DISP_CS -> /DISP_DC
- J5 pad 6: /DISP_DC -> /DISP_DIN
- R44 pad 1: Net-(C67-Pad2) -> /OPAMP_GAIN_VOUT
- R45 pad 2: Net-(U10B-IN+) -> Net-(U9A-IN+)
- U1 pad 153: unconnected-(U2-PG10-Pad153) -> /DPOT_NSHDN
- U1 pad 164: unconnected-(U2-PB6-Pad164) -> /DPOT_SCL
- U1 pad 165: unconnected-(U2-PB7-Pad165) -> /DPOT_SDA
- U1 pad 25: unconnected-(U2-PF7-Pad25) -> Net-(U1-PF7)
- U1 pad 40: unconnected-(U2-PA0-Pad40) -> /UI_ENC_A
- U1 pad 41: Net-(U2-PA1) -> /UI_ENC_B
- U1 pad 43: /MCU_LED_R -> /UI_ENC_SW
- U1 pad 44: /MCU_LED_G -> unconnected-(U1-PH3-Pad44)
- U1 pad 45: /MCU_LED_B -> /UI_SW_A
- U1 pad 46: unconnected-(U2-PH5-Pad46) -> /UI_SW_B
- U1 pad 84: /UI_SW_A -> unconnected-(U1-PH7-Pad84)
- U1 pad 85: /UI_SW_B -> unconnected-(U1-PH8-Pad85)
- U1 pad 86: unconnected-(U2-PH9-Pad86) -> /MCU_LED_R
- U1 pad 87: /UI_ENC_A -> /MCU_LED_G
- U1 pad 88: /UI_ENC_B -> /MCU_LED_B
- U1 pad 89: /UI_ENC_SW -> unconnected-(U1-PH12-Pad89)
- U11 pad 11: /DPOT_P0B -> GND
- U11 pad 13: /DPOT_P0A -> /VREF_+10V
- U4 pad 17: Net-(U8-VREF) -> /OPAMP_VREF
- U7 pad 4: Net-(U6-BST) -> /SMPS_BST
- U9 pad 1: Net-(C57-Pad2) -> Net-(U9A-IN-)
- U9 pad 2: /DAC_IOUT1 -> Net-(U9A-IN-)
- U9 pad 3: GND -> Net-(U9A-IN+)
Routing:
- net +3.3V: track 0.00 -> 151.8 mm, vias 0 -> 12
- net GND: track 0.00 -> 133.4 mm, vias 0 -> 143
- net /POWER_SWITCH_+15V: track 0.00 -> 56.3 mm, vias 0 -> 5
- net /SDRAM_NWE: track 0.00 -> 45.2 mm, vias 0 -> 1
- net /UI_SW_A: track 0.00 -> 43.8 mm
- net /SDRAM.DQ14: track 0.00 -> 42.5 mm, vias 0 -> 1
- net /SDRAM.DQ13: track 0.00 -> 42.4 mm, vias 0 -> 1
- net /SDRAM.DQ15: track 0.00 -> 42.0 mm, vias 0 -> 1
- net /SDRAM_NCS: track 0.00 -> 40.0 mm, vias 0 -> 1
- net /UI_SW_B: track 0.00 -> 38.5 mm
- net /SDRAM_A12: track 0.00 -> 37.5 mm, vias 0 -> 1
- net Net-(Q1-G): track 0.00 -> 35.7 mm
- net /DAC_NCS: track 0.00 -> 34.7 mm, vias 0 -> 2
- net /SD_DAT3: track 0.00 -> 33.8 mm, vias 0 -> 2
- net /SD_DAT2: track 0.00 -> 33.7 mm, vias 0 -> 2
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- added copper zone on F.Cu, net +15V
- added copper zone on B.Cu, net +3.3V
- added copper zone on F.Cu, net +3.3V
- added copper zone on F.Cu, net /CHGPMP_+C
- added copper zone on F.Cu, net /CHGPMP_+LDO
- added copper zone on F.Cu, net /CHGPMP_-C
- added copper zone on F.Cu, net /CHGPMP_-LDO
- added copper zone on F.Cu, net /POWER_SWITCH_+15V
- added copper zone on F.Cu, net /SMPS_BST
- added copper zone on F.Cu, net /SMPS_FB
- added copper zone on F.Cu, net /SMPS_SW
- added copper zone on F.Cu, net /SMPS_VCC
- added copper zone on F.Cu, net /SMPS_VOUT
- added copper zone on F.Cu, net GND
Other:
- board size 341 x 224.6 mm -> 182.7 x 159.8 mm

Commit message: pcb update
Parts:
- added G***: LOGO, LOGO, F.Cu at (367.6, 221.4)
- added J4: BNC_Connector, Connector_Coaxial:SMA_Molex_73251-1153_EdgeMount_Horizontal, F.Cu at (242.2, 217.5)
- moved FID3 228.2 mm to (450.7, 201.5)
- moved FID4 228.2 mm to (450.7, 205.1)
- moved FID5 228.2 mm to (454.3, 201.5)
- moved FID6 228.2 mm to (454.3, 205.1)
- moved H1 228.2 mm to (435.4, 203.8)
- moved H2 228.2 mm to (435.4, 214.0)
- moved H3 228.2 mm to (435.4, 224.1)
- moved H4 228.2 mm to (435.4, 234.3)
- moved TP13 228.2 mm to (458.6, 216.0)
- moved TP14 228.2 mm to (458.6, 220.3)
- moved TP15 228.2 mm to (458.6, 224.7)
- moved TP16 228.2 mm to (458.6, 229.0)
- moved TP5 228.2 mm to (449.9, 216.0)
- moved TP6 228.2 mm to (449.9, 220.3)
- moved TP7 228.2 mm to (449.9, 224.7)
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Routing:
- net +3.3V: track 151.8 -> 283.3 mm, vias 12 -> 22
- net /DPOT_NSHDN: track 0.00 -> 43.8 mm, vias 0 -> 2
- net GND: track 133.4 -> 175.9 mm, vias 143 -> 167
- net /DPOT_SDA: track 4.89 -> 38.7 mm, vias 0 -> 2
- net /DPOT_SCL: track 8.62 -> 36.6 mm, vias 0 -> 2
- net /POWER_SWITCH_+15V: track 56.3 -> 79.7 mm
- net /OPAMP_VREF: track 6.89 -> 29.7 mm
- net /DAC_RFB: track 0.00 -> 20.8 mm
- net /DAC_NCS: track 34.7 -> 15.6 mm
- net /DAC.DB11: track 23.2 -> 5.97 mm
- net /DAC.DB10: track 21.8 -> 5.55 mm
- net /DAC_IOUT1: track 0.00 -> 16.3 mm
- net /DAC.DB9: track 21.5 -> 5.54 mm
- net /DAC.DB8: track 21.6 -> 5.97 mm
- net Net-(U3-Y8): track 20.0 -> 6.56 mm
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- added copper zone on B.Cu, net GND
- added copper zone on In1.Cu, net GND
- added copper zone on In2.Cu, net GND
Other:
- board size 182.7 x 159.8 mm -> 155.9 x 106.6 mm
