File: pcb/direct-digital-synthesis.kicad_sch (KiCad schematic)
At the start: 109 parts, among them IC1 IS45S16800F-7TLA2, J1 TagConnect_TC2030, J2 Micro_SD_Card_Det1, J3 Barrel_Jack_Switch, U1 STM32H723ZGT6, U2 AD5445YCPZ, U3 REF5010AID, U4 LTC3260EDE-PBF, U5 LMR36015FBRNXR, U6 OPA810IDR

Commit message: Updated pcb and src
Parts:
- removed D6: MCU_STATUS_LED_RED, symbol Device:LED
- removed IC1: IS45S16800F-7TLA2, Custom_Memory:SOP80P1176X120-54N, symbol Custom_Memory:IS45S16800F-7TLA2
- removed J2: Micro_SD_Card_Det1, symbol Connector:Micro_SD_Card_Det1
- removed U1: STM32H723ZGT6, Package_QFP:LQFP-144_20x20mm_P0.5mm, symbol MCU_ST_STM32H7:STM32H723ZGTx
- removed U2: AD5445YCPZ, Custom_DACs:CP_20_1_ADI-M, symbol Custom_DACs:AD5445YCPZ
- removed U6: OPA810IDR, Custom_OpAmps:SOIC8_D_TEX-M, symbol Custom_OpAmps:OPA810IDR
- added C19, C21, C22: 1u, Capacitor_SMD:C_0603_1608Metric, symbol Device:C
- added C20: 2u2, Capacitor_SMD:C_0603_1608Metric, symbol Device:C
- added C23, C24, C25, C26, C27: 100n, Capacitor_SMD:C_0603_1608Metric, symbol Device:C
- added IC1: IS42S16160J-7TLI, Custom_Memory:SOP80P1176X120-54N, symbol Custom_Memory:IS42S16160J-7TLI
- added J2: MEM2061-01-188-00-A, Custom_Connectors:MEM20610118800A, symbol Custom_Connectors:MEM2061-01-188-00-A
- added LED1: IN-S66TBTRGB, Custom_LEDs:INS66TBTRGB, symbol Custom_LEDs:IN-S66TBTRGB
- added R10, R11, R12, R13, R14, R15, R16, R21, R23, R24, R25, R26, R27, R28, R30, R31, R32, R33, R34, R35, R36, R6, R8, R9: 22R, Resistor_SMD:R_0603_1608Metric, symbol Device:R
- added R17: 10k, Resistor_SMD:R_0603_1608Metric, symbol Device:R
- added R18, R19, R20: 100R, Resistor_SMD:R_0603_1608Metric, symbol Device:R
- added R22: 0R, Resistor_SMD:R_0603_1608Metric, symbol Device:R
- added R37: 50k, Resistor_SMD:R_0603_1608Metric, symbol Device:R
- added R44, R45: 100k, Resistor_SMD:R_0603_1608Metric, symbol Device:R
- added TP18: MCU_OSC_IN, TestPoint:TestPoint_THTPad_D1.5mm_Drill0.7mm, symbol Connector:TestPoint
- added U1: STM32H750IBT6, Package_QFP:LQFP-176_24x24mm_P0.5mm, symbol MCU_ST_STM32H7:STM32H750IBTx
- added U2, U3: PCHCS541QWRKSRQ1, Custom_LineDrivers:RKS0020B_VQFN_TEX-M, symbol Custom_LineDrivers:PCHCS541QWRKSRQ1
- added U6: AD5445YCPZ, Custom_DACs:CP_20_1_ADI-M, symbol Custom_DACs:AD5445YCPZ
- added U8: OPA810IDR, Custom_OpAmps:SOIC8_D_TEX-M, symbol Custom_OpAmps:OPA810IDR
- added Y1: ECS-2520MVQ-240-BS-TR, Custom_Oscillators:ECS2520MVQ240BSTR, symbol Custom_Oscillators:ECS-2520MVQ-240-BS-TR
- C10: value 100n -> 1u
- C12: value 1u -> 10u; footprint Capacitor_SMD:C_0603_1608Metric -> Capacitor_SMD:C_0805_2012Metric
- C13: value 2u2 -> 1u
- C15: value 2u2 -> 100n
- C18: value 1u -> 2u2
- FID1, FID2, FID3, FID4, FID5, FID6, FID7, H1, H2, H3, H4: now in the parts list
- J3: footprint (none) -> Connector_BarrelJack:BarrelJack_Horizontal
- R5: value 2k2 -> 22R
- renumbered C23 to C28, C28 to C29, C24 to C30, C26 to C31, C19 to C32, C22 to C33, C20 to C34, C25 to C35, C32 to C36, C27 to C37, C34 to C38, C29 to C39, C36 to C40, C21 to C41, C35 to C42, C38 to C43, C33 to C44, C40 to C45, C37 to C46, C30 to C47, C31 to C48, C39 to C49, C41 to C50, C42 to C51, C43 to C52, C44 to C53, C45 to C54, C46 to C55, C47 to C56, C48 to C57, C49 to C58, C50 to C59, C51 to C60, R6 to R29, R10 to R38, R11 to R39, R12 to R40, R13 to R41, R8 to R42, R9 to R43, U3 to U5, U5 to U7
Connections:
- net +12V: now also U8.7 (VS+)
- net +3.3V: now also C10.1, C13.1, C19.1, C21.1, C22.1, C24.1, C25.1, C26.1, C27.1, IC1.1 (VDD_1), IC1.14 (VDD_2), IC1.27 (VDD_3), IC1.3 (VDDQ_1), IC1.43 (VDDQ_3), IC1.49 (VDDQ_4), IC1.9 (VDDQ_2), J2.P4 (VDD), LED1.1 (COM+), R17.1, U1.103 (VDD), U1.114 (VDD33_USB), U1.127 (VDD), U1.136 (VDD), U1.149 (VDD), U1.15 (VDD), U1.159 (VDD), U1.171 (PDR_ON), U1.172 (VDD), U1.23 (VDD), U1.36 (VDD), U1.38 (VREF+), U1.39 (VDDA), U1.49 (VDD), U1.6 (VBAT), U1.62 (VDD), U1.72 (VDD), U1.82 (VDD), U1.91 (VDD), U2.20 (VCC), U3.20 (VCC), U6.16 (VDD), Y1.4 (VDD); no longer C18.1
- net -12V: now also U8.4 (VS-)
- net DAC_IOUT1: now also U6.19 (IOUT1), U8.2 (VIN-)
- net DAC_NCS: now also R24.2, U6.14 (CS*)
- net DAC_RFB: now also R44.2, R45.1, U6.18 (RFB)
- net GND: now also C19.2, C20.2, C21.2, C22.2, C23.2, C24.2, C25.2, C26.2, C27.2, IC1.12 (VSSQ_2), IC1.28 (VSS_1), IC1.41 (VSS_2), IC1.46 (VSSQ_3), IC1.52 (VSSQ_4), IC1.54 (VSS_3), IC1.6 (VSSQ_1), J2.CD2 (CARD_DETECT_2), J2.G1 (GND_1), J2.G2 (GND_2), J2.P6 (VSS), R45.2, U1.102 (VSS), U1.113 (VSS), U1.126 (VSS), U1.135 (VSS), U1.14 (VSS), U1.148 (VSS), U1.158 (VSS), U1.166 (BOOT0), U1.22 (VSS), U1.37 (VSSA), U1.48 (VSS), U1.61 (VSS), U1.71 (VSS), U1.90 (VSS), U2.1 (*OE1), U2.10 (GND), U2.19 (*OE2), U2.21 (GND), U2.3 (A2), U2.4 (A3), U2.5 (A4), U3.1 (*OE1), U3.10 (GND), U3.19 (*OE2), U3.21 (GND), U6.1 (GND), U6.15 (R/W*), U6.20 (IOUT2), U6.21 (EP), U8.3 (VIN+), Y1.2 (GND); no longer R5.2
- net MCU_NRST: now also C15.1, U1.31 (NRST); no longer C10.1
- net MCU_SWCLK: now also U1.137 (PA14)
- net MCU_SWDIO: now also U1.124 (PA13)
- net MCU_SWO: now also U1.161 (PB3)
- net SDRAM_A0: now also IC1.23 (A0), U1.16 (PF0)
- net SDRAM_A1: now also IC1.24 (A1), U1.17 (PF1)
- net SDRAM_A10: now also IC1.22 (A10), U1.66 (PG0)
- net SDRAM_A11: now also IC1.35 (A11), U1.67 (PG1)
- net SDRAM_A2: now also IC1.25 (A2), U1.18 (PF2)
- net SDRAM_A3: now also IC1.26 (A3), U1.19 (PF3)
- net SDRAM_A4: now also IC1.29 (A4), U1.20 (PF4)
- net SDRAM_A5: now also IC1.30 (A5), U1.21 (PF5)
- net SDRAM_A6: now also IC1.31 (A6), U1.60 (PF12)
- net SDRAM_A7: now also IC1.32 (A7), U1.63 (PF13)
- net SDRAM_A8: now also IC1.33 (A8), U1.64 (PF14)
- net SDRAM_A9: now also IC1.34 (A9), U1.65 (PF15)
- net SDRAM_BA0: now also IC1.20 (BA0), U1.108 (PG4)
- net SDRAM_BA1: now also IC1.21 (BA1), U1.109 (PG5)
- net SDRAM_CKE: now also IC1.37 (CKE), U1.35 (PC3_C)
- net SDRAM_CLK: now also IC1.38 (CLK), U1.112 (PG8)
- net SDRAM_DQMH: now also IC1.39 (DQMH), U1.170 (PE1)
- net SDRAM_DQML: now also IC1.15 (DQML), U1.169 (PE0)
- net SDRAM_NCAS: now also IC1.17 (~{CAS}), U1.160 (PG15)
- net SDRAM_NCS: now also IC1.19 (~{CS}), U1.34 (PC2_C)
- net SDRAM_NRAS: now also IC1.18 (~{RAS}), U1.59 (PF11)
- net SDRAM_NWE: now also IC1.16 (~{WE}), U1.32 (PC0)
- net VREF_+10V: now also R37.2
- net at R29.1: now also U3.18 (Y1)
- net DAC.DB7: now reaches R29.2
- net DAC.DB7: now also U6.6 (DB7)
- net at R5.1: now also U1.131 (PI0)
- net at R7.1: now also U1.133 (PI2)
- net MCU_DAC.DB2: now reaches R7.2
- net MCU_DAC.DB2: now also U3.7 (A6)
- new net: R34.1, U3.13 (Y6)
- new net: R36.1, U3.11 (Y8)
- new net: R16.1, U1.13 (PI11)
- new net: R8.1, U1.134 (PI3)
- new net: R35.1, U3.12 (Y7)
- new net: R24.1, U2.18 (Y1)
- new net: LED1.2 (K_RED), R18.1
- new net: LED1.3 (K_BLUE), R20.1
- new net: LED1.4 (K_GREEN), R19.1
- new net: R32.1, U3.15 (Y4)
- new net: R15.1, U1.12 (PI10)
- new net: R22.1, U1.141 (PC12)
- new net: R26.1, U2.13 (Y6)
- new net: R23.1, Y1.3 (OUTPUT)
- new net: R37.1, U6.17 (VREF)
- new net: R28.1, U2.11 (Y8)
- new net: R27.1, U2.12 (Y7)
- new net: R25.1, U2.14 (Y5)
- new net: R13.1, U1.7 (PI8)
- new net: R33.1, U3.14 (Y5)
- new net: R11.1, U1.175 (PI6)
- new net: C18.1, U1.81 (VCAP)
- new net: R31.1, U3.16 (Y3)
- new net: R14.1, U1.11 (PI9)
- new net: R30.1, U3.17 (Y2)
- new net: R6.1, U1.132 (PI1)
- new net: R10.1, U1.174 (PI5)
- new net: C20.1, U1.125 (VCAP)
- new net: R9.1, U1.173 (PI4)
- new net: R12.1, U1.176 (PI7)
- new net: R21.1, U1.41 (PA1)
- new net DAC.DB0: R36.2, U6.13 (DB0)
- new net DAC.DB1: R35.2, U6.12 (DB1)
- new net DAC.DB10: R26.2, U6.3 (DB10)
- new net DAC.DB11: R25.2, U6.2 (DB11)
- new net DAC.DB2: R34.2, U6.11 (DB2)
- new net DAC.DB3: R33.2, U6.10 (DB3)
- new net DAC.DB4: R32.2, U6.9 (DB4)
- new net DAC.DB5: R31.2, U6.8 (DB5)
- new net DAC.DB6: R30.2, U6.7 (DB6)
- new net DAC.DB8: R28.2, U6.5 (DB8)
- new net DAC.DB9: R27.2, U6.4 (DB9)
- new net MCU_DAC.DB0: R5.2, U3.9 (A8)
- new net MCU_DAC.DB1: R6.2, U3.8 (A7)
- new net MCU_DAC.DB10: R15.2, U2.7 (A6)
- new net MCU_DAC.DB11: R16.2, U2.6 (A5)
- new net MCU_DAC.DB3: R8.2, U3.6 (A5)
- new net MCU_DAC.DB4: R9.2, U3.5 (A4)
- new net MCU_DAC.DB5: R10.2, U3.4 (A3)
- new net MCU_DAC.DB6: R11.2, U3.3 (A2)
- new net MCU_DAC.DB7: R12.2, U3.2 (A1)
- new net MCU_DAC.DB8: R13.2, U2.9 (A8)
- new net MCU_DAC.DB9: R14.2, U2.8 (A7)
- new net MCU_DAC_NCS: R21.2, U2.2 (A1)
- new net MCU_LED_B: R20.2, U1.45 (PH4)
- new net MCU_LED_G: R19.2, U1.44 (PH3)
- new net MCU_LED_R: R18.2, U1.43 (PH2)
- new net MCU_OSC_IN: R23.2, TP18.1, U1.29 (PH0)
- new net OPAMP_VOUT: R44.1, U8.6 (VO)
- new net SDRAM.DQ0: IC1.2 (DQ0), U1.104 (PD14)
- new net SDRAM.DQ1: IC1.4 (DQ1), U1.105 (PD15)
- new net SDRAM.DQ10: IC1.45 (DQ10), U1.76 (PE13)
- new net SDRAM.DQ11: IC1.47 (DQ11), U1.77 (PE14)
- new net SDRAM.DQ12: IC1.48 (DQ12), U1.78 (PE15)
- new net SDRAM.DQ13: IC1.50 (DQ13), U1.96 (PD8)
- new net SDRAM.DQ14: IC1.51 (DQ14), U1.97 (PD9)
- new net SDRAM.DQ15: IC1.53 (DQ15), U1.98 (PD10)
- new net SDRAM.DQ2: IC1.5 (DQ2), U1.142 (PD0)
- new net SDRAM.DQ3: IC1.7 (DQ3), U1.143 (PD1)
- new net SDRAM.DQ4: IC1.8 (DQ4), U1.68 (PE7)
- new net SDRAM.DQ5: IC1.10 (DQ5), U1.69 (PE8)
- new net SDRAM.DQ6: IC1.11 (DQ6), U1.70 (PE9)
- new net SDRAM.DQ7: IC1.13 (DQ7), U1.73 (PE10)
- new net SDRAM.DQ8: IC1.42 (DQ8), U1.74 (PE11)
- new net SDRAM.DQ9: IC1.44 (DQ9), U1.75 (PE12)
- new net SDRAM_A12: IC1.36 (A12), U1.106 (PG2)
- new net SD_CLK: J2.P5 (CLK), R22.2
- new net SD_CMD: J2.P3 (CMD), U1.144 (PD2)
- new net SD_DAT0: J2.P7 (DAT0), U1.117 (PC8)
- new net SD_DAT1: J2.P8 (DAT1), U1.118 (PC9)
- new net SD_DAT2: J2.P1 (DAT2), U1.139 (PC10)
- new net SD_DAT3: J2.P2 (CD/DAT3), U1.140 (PC11)
- new net SD_NCD: C23.1, J2.CD1 (CARD_DETECT_1), R17.2, U1.145 (PD3)
- no-connect marks 7 -> 9
Other:
- note added: "1/8W rated current limiting resistors"
- note added: "256Mb (16Mx16), 143MHz SDRAM"
- note added: "Clock Oscillator"
- note added: "Display"
- note added: "Find correct value of pull up resistor for SD_NCD"
- note added: "Gain=(100k+100k)/100k=2 (Pg 21)"
- note added: "No termination resistors on the SDRAM lines since SDRAM and MCU are placed closed to each other. Might have to consider length matching depending on speed of SDRAM. CAS Latency of 2 selected -> Running clock at max, 133 MHz In CubeIDE select SDRAM common clock to 3 clock cycles which then divides the FMC clock running at 240 MHz by 3. Therefore the SDRAM is running at effectively 80 MHz. This fal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"
- note added: "POTENTIALLY ADD SWITCH HERE TO RESET MCU NRST"
- note added: "Place series termination resistors close to the driver output"
- note added: "Power Switch"
- note added: "Read functionality is essentially disabled since the Schmitt Triggers Buffers are unidirectional. Therefore tie R/~{W} to GND which fixes the DAC mode to be write only."
- note added: "Relying on internal pull up resistors and ESD protection of STM32 MCU SD Clock Running at 40 MHz"
- note added: "Status LED"
- note added: "Unused inputs must be tied either to VCC or GND. Unused outputs must be no connects. (Pg 12)"
- note removed: "128Mb (8Mx16), 143MHz SDRAM"
- note removed: "Add series termination resistors to CLK and WRT lines to reduce overshoot and ringing"
- note removed: "Clock Oscillators"
- note removed: "DC Input Power Jack (Connects to wall wart)"
- note removed: "IOUT2 and the exposed pad must be connected to AGND (Pg 9)"
- note removed: "Low Noise Dual Supply Inverting Charge Pump (+-12VDC)"
- note removed: "No termination resistors on the SDRAM lines since SDRAM and MCU are placed closed to each other"
- note removed: "POTENTAILLY ADD SWITCH HERE TO RESET MCU NRST"
- note removed: "Precision Voltage Reference"
- note removed: "Relying on internal pull up resistors and ESD protection of STM32 MCU SDMMC Running at 90 MHz"
- note removed: "SMPS (3.3VDC)"
- moved on the sheet: C28, C29, C30, C31, C32, C33, C34, C35, C36, C37, C38, C39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

Commit message: pcb update
Parts:
- removed C47, C48: 100n, Capacitor_SMD:C_0603_1608Metric, symbol Device:C
- removed R17: 10k, Resistor_SMD:R_0603_1608Metric, symbol Device:R
- removed R44: 100k, Resistor_SMD:R_0603_1608Metric, symbol Device:R
- removed U8: OPA810IDR, Custom_OpAmps:SOIC8_D_TEX-M, symbol Custom_OpAmps:OPA810IDR
- added C2, C49, C50: 100n, Capacitor_SMD:C_0603_1608Metric, symbol Device:C
- added D2, D6: D_TVS, symbol Device:D_TVS
- added J4: Conn_Coaxial, symbol Connector:Conn_Coaxial
- added Q1: PMOS, symbol Simulation_SPICE:PMOS
- added R1, R46: 10k, Resistor_SMD:R_0603_1608Metric, symbol Device:R
- added R18: 50k, Resistor_SMD:R_0603_1608Metric, symbol Device:R
- added R47, R48: 20k, Resistor_SMD:R_0603_1608Metric, symbol Device:R
- added SW1: SW_DPDT_x2, symbol Switch:SW_DPDT_x2
- added U8: OPA2810IDGKR, Custom_OpAmps:DGK0008A_N, symbol Custom_OpAmps:OPA2810IDGKR
- R45: value 100k -> 20k
- renumbered C9 to C10, C10 to C11, C11 to C12, C12 to C13, C13 to C14, C14 to C15, C15 to C16, C16 to C17, C17 to C18, C18 to C19, C19 to C20, C20 to C21, C21 to C22, C22 to C23, C23 to C24, C24 to C25, C25 to C26, C26 to C27, C27 to C28, C28 to C29, C2 to C3, C29 to C30, C30 to C31, C31 to C32, C32 to C34, C34 to C36, C36 to C37, C37 to C38, C38 to C39, C3 to C4, C39 to C40, C40 to C41, C41 to C42, C42 to C43, C43 to C44, C44 to C45, C45 to C46, C46 to C47, C49 to C48, C4 to C5, C50 to C51, C51 to C52, C52 to C53, C53 to C54, C54 to C55, C55 to C56, C56 to C57, C57 to C58, C58 to C59, C5 to C6, C59 to C60, C60 to C61, C6 to C7, C7 to C8, C8 to C9, D2 to D3, D3 to D4, D4 to D5, D5 to D7, R9 to R10, R10 to R11, R11 to R12, R12 to R13, R13 to R14, R14 to R15, R15 to R16, R16 to R17, R18 to R19, R1 to R2, R19 to R20, R20 to R21, R21 to R22, R22 to R23, R23 to R24, R24 to R25, R25 to R26, R26 to R27, R27 to R28, R28 to R29, R2 to R3, R29 to R30, R30 to R31, R31 to R32, R32 to R33, R33 to R34, R34 to R35, R35 to R36, R36 to R37, R37 to R38, R38 to R39, R3 to R4, R39 to R40, R40 to R41, R41 to R42, R42 to R43, R43 to R44, R4 to R5, R5 to R6, R6 to R7, R7 to R8, R8 to R9
Connections:
- net +12V: now also C49.1, U8.8 (V+)
- net +15V: now also C2.1, D2.2 (A2), Q1.3 (S), R1.1
- net +3.3V: now also R18.2
- net -12V: now also C50.2, U8.4 (V-)
- net DAC_IOUT1: now also U8.2 (IN-)
- net GND: now also C49.2, C50.1, D2.1 (A1), D6.1 (A1), J4.2 (Ext), SW1.3 (C), U8.3 (IN+), U8.5 (IN+); no longer R45.2
- net OPAMP_VOUT: now also J4.1 (In), R48.2, U8.7
- net VREF_+10V: now also R47.2
- net SD_NCD renamed SD_CD
- net SD_CD: now also R18.1
- new net: C2.2, Q1.2 (G), R1.2, SW1.2 (B)
- new net: R45.2, R46.1, U8.1
- new net: R46.2, R47.1, R48.1, U8.6 (IN-)
- new net POWER_SWITCH: D6.2 (A2), Q1.1 (D)
- no-connect marks 9 -> 13
Other:
- note added: "50 Ohm BNC Connector"
- note added: "Connector for external display"
- note added: "Display Connector"
- note added: "High side PMOS Enhancement Mode MOSFET rather then a mechanical power switch to switch on/off power supply to limit inrush current and thus sparking."
- note added: "Inverting Amplifier Gain = -(20k/10k) = -2"
- note added: "Make sure that PMOS has low R_{DS-on} and enough continuous I_{D} rating to handle total current draw. Also make sure to check maximum V_{gs} rating and see if it can handle -15VDC"
- note added: "When SD card is inserted SD_CD is high and when SD card is not inserted SD_CD is low"
- note removed: "Display"
- note removed: "Find correct value of pull up resistor for SD_NCD"
- note removed: "Gain=(100k+100k)/100k=2 (Pg 21)"
- moved on the sheet: C34, C36, C42, C53, C54, C55, C56, C57, C58, C59, C60, C61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

Commit message: pcb update
Parts:
- removed Q1: PMOS, symbol Simulation_SPICE:PMOS
- added Q1: PMPB27EPZ, Custom_MOSFETs:DFN-2020MD-6, symbol Custom_MOSFETs:PMPB27EPZ
Connections:
- net +15V: now also Q1.4 (S), Q1.8 (S)
- net POWER_SWITCH: now also Q1.1 (D), Q1.2 (D), Q1.5 (D), Q1.6 (D), Q1.7 (D)
- net at C2.2, R1.2, SW1.2 (B): now also Q1.3 (G)
Changed lines of the file:
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@@
 	)
 	(symbol
-		(lib_id "Simulation_SPICE:PMOS")
-		(at 101.6 660.4 270)
-		(mirror x)
-		(unit 1)
-		(exclude_from_sim no)
-		(in_bom yes)
-		(on_board yes)
-		(dnp no)
-		(property "Reference" "Q1"
-			(at 101.6 651.51 90)
-			(effects
-				(font
-					(size 1.27 1.27)
-				)
-			)
-		)
-		(property "Value" "PMOS"
-			(at 101.6 654.05 90)
-			(effects
-				(font
-					(size 1.27 1.27)
-				)
-			)
-		)
-		(property "Footprint" ""
-			(at 104.14 655.32 0)
-			(effects
-				(font
-					(size 1.27 1.27)
-				)
-				(hide yes)
-			)
-		)
-		(property "Datasheet" "https://ngspice.sourceforge.io/docs/ngspice-html-manual/manual.xhtml#cha_MOSFETs"
-			(at 88.9 660.4 0)
-			(effects
-				(font
-					(size 1.27 1.27)
-				)
-				(hide yes)
-			)
-		)
-		(property "Description" "P-MOSFET transistor, drain/source/gate"
-			(at 101.6 660.4 0)
-			(effects
-				(font
-					(size 1.27 1.27)
-				)
-				(hide yes)
-			)
-		)
-		(property "Sim.Device" "PMOS"
-			(at 84.455 660.4 0)
-			(effects
-				(font
-					(size 1.27 1.27)
-				)
-				(hide yes)
-			)
-		)
-		(property "Sim.Type" "VDMOS"
-			(at 82.55 660.4 0)
-			(effects
-				(font
-					(size 1.27 1.27)
-				)
-				(hide yes)
-			)
-		)
-		(property "Sim.Pins" "1=D 2=G 3=S"
-			(at 86.36 660.4 0)
-			(effects
-				(font
-					(size 1.27 1.27)
-				)
-				(hide yes)
-			)
-		)
-		(pin "3"
-		)
-		(pin "1"
-		)
-		(pin "2"
-		)
-		(instances
-			(project "direct-digital-synthesis"
-				(path "/9fa233b0-8355-46f9-8752-6afcf092d80a"
-					(reference "Q1")
-					(unit 1)
-				)
-			)
-		)
-	)
-	(symbol
 		(lib_id "power:GND")
 		(at 610.87 539.75 0)
@@
 					(unit 1)
 				)
+			)
+		)
+	)
+	(symbol
+		(lib_id "Custom_MOSFETs:PMPB27EPZ")
+		(at 106.68 659.13 270)
+		(mirror x)
+		(unit 1)
+		(exclude_from_sim no)
+		(in_bom yes)
+		(on_board yes)
+		(dnp no)
+		(property "Reference" "Q1"
+			(at 101.6 651.51 90)
+			(effects
+				(font
+					(size 1.27 1.27)
+				)
+			)
+		)
+		(property "Value" "PMPB27EPZ"
+			(at 101.6 654.05 90)
+			(effects
+				(font
+					(size 1.27 1.27)
+				)
+			)
+		)
+		(property "Footprint" "Custom_MOSFETs:DFN-2020MD-6"
+			(at 88.646 659.13 0)
+			(effects
+				(font
+					(size 1.27 1.27)
+				)
+				(hide yes)
+			)
+		)
+		(property "Datasheet" ""
+			(at 116.332 659.13 0)
+			(effects
+				(font
+					(size 1.27 1.27)
+				)
+				(hide yes)
+			)
+		)
+		(property "Description" "30V, Single P-channel Trench MOSFET"
+			(at 60.96 658.368 0)
+			(effects
+				(font
+					(size 1.27 1.27)
+				)
+				(hide yes)
+			)
+		)
+		(property "Manufacturer_Name" "Nexperia"
+			(at 55.626 658.876 0)
+			(effects
+				(font
+					(size 1.27 1.27)
+				)
+				(hide yes)
+			)
+		)
+		(property "Mouser Part Number" "771-PMPB27EPZ"
+			(at 51.562 658.876 0)
+			(effects
+				(font
+					(size 1.27 1.27)
+				)
+				(hide yes)
+			)
+		)
+		(pin "7"
+		)
+		(pin "1"
+		)
+		(pin "2"
+		)
+		(pin "8"
+		)
+		(pin "4"
+		)
+		(pin "6"
+		)
+		(pin "3"
+		)
+		(pin "5"
+		)
+		(instances
+			(project ""
+				(path "/9fa233b0-8355-46f9-8752-6afcf092d80a"
+					(reference "Q1")
+					(unit 1)
+				)

Commit message: update pcb
Parts:
- removed C43: 10u, Capacitor_SMD:C_0805_2012Metric, symbol Device:C
- removed D1, D3, D4, D5, D7: Zener, symbol Device:D_Zener
- removed L1: 10u, symbol Device:L
- removed R46: 10k, Resistor_SMD:R_0603_1608Metric, symbol Device:R
- removed R47, R48: 20k, Resistor_SMD:R_0603_1608Metric, symbol Device:R
- removed U2: PCHCS541QWRKSRQ1, Custom_LineDrivers:RKS0020B_VQFN_TEX-M, symbol Custom_LineDrivers:PCHCS541QWRKSRQ1
- removed U7: LMR36015FBRNXR, Custom_PowerModules:RNX0012B, symbol Custom_PowerModules:LMR36015FBRNXR
- removed U8: OPA2810IDGKR, Custom_OpAmps:DGK0008A_N, symbol Custom_OpAmps:OPA2810IDGKR
- added C1, C20, C25, C28, C29, C30, C71, C72, C79, C80, C81: 100n, Capacitor_SMD:C_0603_1608Metric, symbol Device:C
- added C49, C58, C59, C68, C69: 10u, Capacitor_SMD:C_0805_2012Metric, symbol Device:C
- added C57: 4p7, Capacitor_SMD:C_0603_1608Metric, symbol Device:C
- added C66, C67: 430p, Capacitor_SMD:C_0603_1608Metric, symbol Device:C
- added C77: 120p, Capacitor_SMD:C_0603_1608Metric, symbol Device:C
- added C78: 1n8, Capacitor_SMD:C_0603_1608Metric, symbol Device:C
- added J2: Conn_01x07_Socket, Connector_PinSocket_2.54mm:PinSocket_1x07_P2.54mm_Vertical, symbol Connector:Conn_01x07_Socket
- added JP1, JP2, JP3, JP4, JP5: Power_Jumper, symbol Jumper:Jumper_2_Open
- added L1: 6u8, Custom_Inductors:ASPIAIG-F6060, symbol Custom_Inductors:ASPIAIG-F6060-6R8M-T
- added R18, R21, R22, R24, R53: 10k, Resistor_SMD:R_0603_1608Metric, symbol Device:R
- added R19: 50k, Resistor_SMD:R_0603_1608Metric, symbol Device:R
- added R26, R27: 22R, Resistor_SMD:R_0603_1608Metric, symbol Device:R
- added R54: 20k, Resistor_SMD:R_0603_1608Metric, symbol Device:R
- added R55: 75R, Resistor_SMD:R_0603_1608Metric, symbol Device:R
- added R56: 365R, Resistor_SMD:R_0603_1608Metric, symbol Device:R
- added R57: 442R, Resistor_SMD:R_0603_1608Metric, symbol Device:R
- added R58: 887R, Resistor_SMD:R_0603_1608Metric, symbol Device:R
- added R59: 84R5, Resistor_SMD:R_0603_1608Metric, symbol Device:R
- added R60: 158R, Resistor_SMD:R_0603_1608Metric, symbol Device:R
- added SW1, SW2: SW_Push, Button_Switch_THT:SW_PUSH_6mm, symbol Switch:SW_Push
- added TP19: POWER_+15V, TestPoint:TestPoint_Keystone_5000-5004_Miniature, symbol Connector:TestPoint
- added TP20: POWER_+10V, TestPoint:TestPoint_Keystone_5000-5004_Miniature, symbol Connector:TestPoint
- added TP21: POWER_-12V, TestPoint:TestPoint_Keystone_5000-5004_Miniature, symbol Connector:TestPoint
- added TP22: POWER_+12V, TestPoint:TestPoint_Keystone_5000-5004_Miniature, symbol Connector:TestPoint
- added TP23: POWER_+3V3, TestPoint:TestPoint_Keystone_5000-5004_Miniature, symbol Connector:TestPoint
- added U1: PEC12R-3225F-S0024, Custom_Encoders:PEC12R3225FS0024, symbol Custom_Encoders:PEC12R-3225F-S0024
- added U10, U9: AD8066ARZ-R7, Custom_OpAmps:R_8_ADI-M, symbol Custom_OpAmps:AD8066ARZ-R7
- added U11: MCP45HV51-ST, Package_SO:TSSOP-14_4.4x5mm_P0.65mm, symbol Potentiometer_Digital:MCP45HV51-ST
- added U4: PCHCS541QWRKSRQ1, Custom_LineDrivers:RKS0020B_VQFN_TEX-M, symbol Custom_LineDrivers:PCHCS541QWRKSRQ1
- added U6: LMR36015FBRNXR, Custom_PowerModules:RNX0012B, symbol Custom_PowerModules:LMR36015FBRNXR
- R23: value 0R -> 10k
- R45: renamed from R38; value 50k -> 0R
- R52: renamed from R45; value 20k -> 0R
- TP1, TP18: footprint TestPoint:TestPoint_THTPad_D1.5mm_Drill0.7mm -> TestPoint:TestPoint_Keystone_5000-5004_Miniature
- renumbered C9 to C10, C24 to C11, C10 to C12, C11 to C13, C12 to C14, C14 to C15, C15 to C16, C26 to C17, C16 to C18, C17 to C19, C13 to C2, C18 to C21, C19 to C22, C20 to C23, C21 to C24, C22 to C26, C23 to C27, C1 to C3, C25 to C31, C27 to C32, C28 to C33, C33 to C34, C29 to C35, C35 to C36, C38 to C37, C30 to C38, C40 to C39, C3 to C4, C31 to C40, C32 to C41, C2 to C42, C34 to C43, C36 to C44, C37 to C45, C45 to C46, C39 to C47, C41 to C48, C4 to C5, C42 to C50, C47 to C51, C44 to C52, C48 to C53, C46 to C54, C51 to C55, C52 to C56, C5 to C6, C49 to C60, C50 to C61, C53 to C62, C54 to C63, C55 to C64, C56 to C65, C6 to C7, C57 to C70, C58 to C73, C59 to C74, C60 to C75, C61 to C76, C7 to C8, C8 to C9, D2 to D1, D6 to D2, J2 to J1, J1 to J3, J3 to J4, J4 to J5, R18 to R1, R24 to R20, R22 to R25, R19 to R28, R20 to R29, R21 to R30, R25 to R31, R26 to R32, R27 to R33, R28 to R34, R29 to R35, R30 to R36, R31 to R37, R32 to R38, R33 to R39, R34 to R40, R35 to R41, R36 to R42, R37 to R43, R1 to R44, R43 to R46, R44 to R47, R39 to R48, R40 to R49, R41 to R50, R42 to R51, SW1 to SW3, U1 to U2, U4 to U5, U5 to U7, U6 to U8
Connections:
- net +12V: now also C58.1, C68.1, C71.1, C81.1, JP4.2 (B), U10.8 (V+), U11.14 (V+), U9.8 (V+); no longer C54.1, R50.1, U5.10 (LDO+)
- net +15V: no longer C34.1, C35.1, C36.2, C37.2, C40.1, U5.1 (EN+), U5.11 (EN-), U5.9 (VIN), U7.2 (VIN)
- net +3.3V: now also C1.2, C79.1, J2.1 (Pin_1), JP5.2 (B), R19.2, R21.2, R22.2, U11.1 (VL), U4.20 (VCC); no longer C51.2, C53.1, C55.1, C56.2, R46.1
- net -12V: now also C59.2, C69.2, C72.2, C80.2, JP3.2 (B), U10.4 (V-), U11.10 (V-), U9.4 (V-); no longer C52.1, R48.1, U5.5 (LDO-)
- net DAC_IOUT1: now also C57.1, U9.2 (IN-)
- net GND: now also U3.3 (A2), U3.4 (A3), U3.5 (A4), C1.1, C20.2, C25.2, C28.2, C29.2, C30.2, C49.2, C58.2, C59.1, C66.2, C68.2, C69.1, C71.2, C72.1, C77.2, C79.2, C80.1, C81.2, J2.2 (Pin_2), R57.1, SW1.1, SW2.1, U1.2, U1.C1, U11.3 (A1), U11.5 (A0), U11.6 (~{WLAT}), U11.9 (DGND), U4.1 (*OE1), U4.10 (GND), U4.19 (*OE2), U4.21 (GND), U6.1 (PGND), U6.11 (PGND), U6.6 (AGND), U6.8 (PG), U9.3 (IN+)
- net MCU_DAC.DB0: now also U4.9 (A8); no longer U3.9 (A8)
- net MCU_DAC.DB1: now also U4.8 (A7); no longer U3.8 (A7)
- net MCU_DAC.DB10: now also U3.7 (A6)
- net MCU_DAC.DB11: now also U3.6 (A5)
- net MCU_DAC.DB2: now also U4.7 (A6); no longer U3.7 (A6)
- net MCU_DAC.DB3: now also U4.6 (A5); no longer U3.6 (A5)
- net MCU_DAC.DB4: now also U4.5 (A4); no longer U3.5 (A4)
- net MCU_DAC.DB5: now also U4.4 (A3); no longer U3.4 (A3)
- net MCU_DAC.DB6: now also U4.3 (A2); no longer U3.3 (A2)
- net MCU_DAC.DB7: now also U4.2 (A1); no longer U3.2 (A1)
- net MCU_DAC.DB8: now also U3.9 (A8)
- net MCU_DAC.DB9: now also U3.8 (A7)
- net MCU_DAC_NCS: now also U3.2 (A1)
- net SD_CLK: now also R27.2; no longer R23.2
- net VREF_+10V: now also JP2.2 (B), R54.2; no longer U7.6 (VOUT)
- net at R36.1: now also U4.18 (Y1); no longer U3.18 (Y1)
- net at C46.2: now also L1.1, U6.12 (SW), U6.3 (NC)
- net at C46.1: now also U6.4 (BST)
- net at C39.1: now also U6.5 (VCC)
- net at C51.1, R46.2, R47.1: now also U6.7 (FB)
- net at R41.1: now also U4.13 (Y6); no longer U3.13 (Y6)
- net at R43.1: now also U4.11 (Y8); no longer U3.11 (Y8)
- net at R52.2: now also C57.2, R53.1, U9.1
- net at R42.1: now also U4.12 (Y7); no longer U3.12 (Y7)
- net at R31.1: now also U3.18 (Y1)
- net at R39.1: now also U4.15 (Y4); no longer U3.15 (Y4)
- net at R23.1: now also R21.1, U1.A1; no longer U2.141 (PC12)
- net at R33.1: now also U3.13 (Y6)
- net at R35.1: now also U3.11 (Y8)
- net at R34.1: now also U3.12 (Y7)
- net at R32.1: now also U3.14 (Y5)
- net at R40.1: now also U4.14 (Y5); no longer U3.14 (Y5)
- net at U3.16 (Y3): no longer R38.1
- net at U3.17 (Y2): no longer R37.1
- net DISP_CS: now reaches U2.50 (PA4)
- net DISP_CS: now also J2.5 (Pin_5)
- net at U2.51 (PA5): now also R26.1
- net DISP_DC: now reaches U2.52 (PA6)
- net DISP_DC: now also J2.6 (Pin_6)
- net DISP_DIN: now reaches U2.53 (PA7)
- net DISP_DIN: now also J2.3 (Pin_3)
- net DISP_NRST: now reaches U2.54 (PC4)
- net DISP_NRST: now also J2.7 (Pin_7)
- net UI_SW_A: now reaches U2.84 (PH7)
- net UI_SW_A: now also C25.1, SW1.2
- net UI_SW_B: now reaches U2.85 (PH8)
- net UI_SW_B: now also C28.1, SW2.2
- net UI_ENC_A: now reaches U2.87 (PH10)
- net UI_ENC_A: now also R23.2, C29.1
- net UI_ENC_B: now reaches U2.88 (PH11)
- net UI_ENC_B: now also C30.1, R24.2
- net UI_ENC_SW: now reaches U2.89 (PH12)
- net UI_ENC_SW: now also C20.1, R18.1
- net OPAMP_VOUT renamed OPAMP_VOUT_FILT
- net OPAMP_VOUT_FILT: now also C78.2, U10.6 (IN-), U10.7
- net POWER_SWITCH renamed PMOS_DRAIN
- net PMOS_DRAIN: now also JP1.1 (A), TP19.1
- new net: C78.1, R59.2, R60.1
- new net: C77.1, R60.2, U10.5 (IN+)
- new net: C67.1, R55.2, R56.1
- new net: C54.1, JP4.1 (A), R50.1, TP22.1, U5.10 (LDO+)
- new net: C51.2, C53.1, C55.1, C56.2, JP5.1 (A), L1.2, R46.1, TP23.1
- new net: R18.2, R19.1, U1.1
- new net: C52.1, JP3.1 (A), R48.1, TP21.1, U5.5 (LDO-)
- new net: C67.2, R58.2, R59.1, U10.1
- new net: C66.1, R56.2, U10.3 (IN+)
- new net: C49.1, JP2.1 (A), TP20.1, U7.6 (VOUT)
- new net: R22.1, R24.1, U1.B1
- new net: R57.2, R58.1, U10.2 (IN-)
- new net: R53.2, R54.1, U9.5 (IN+)
- new net: R38.1, U4.16 (Y3)
- new net: R27.1, U2.141 (PC12)
- new net: R37.1, U4.17 (Y2)
- new net DISP_CLK: J2.4 (Pin_4), R26.2
- new net DPOT_NSHDN: U11.8 (~{SHDN})
- new net DPOT_P0A: U11.13 (P0A)
- new net DPOT_P0B: U11.11 (P0B)
- new net DPOT_P0W: U11.12 (P0W)
- new net DPOT_SCL: U11.2 (SCL)
- new net DPOT_SDA: U11.4 (SDA)
- new net OPAMP_DC_BIAS_VOUT: R55.1, U9.6 (IN-), U9.7
- new net POWER_SWITCH_+15V: C34.1, C35.1, C36.2, C37.2, C40.1, JP1.2 (B), U5.1 (EN+), U5.11 (EN-), U5.9 (VIN), U6.10 (VIN), U6.2 (VIN), U6.9 (EN), U7.2 (VIN)
- no-connect marks 13 -> 80
Other:
- note added: "At full white screen pulls about 60mA"
- note added: "DC Bias"
- note added: "Digital Potentiometer"
- note added: "I2C Device Address is 0111 100b (Pg 51)"
- note added: "Match specific trace width and board layer thickness to get 50 Ohm characteristic impedance. JLCPCB provides impedance calculator"
- note added: "Need a fast slew rate op amp for ouput signal since output peak to peak voltage is large. For a sin wave, slew rate=A_{pp}*2π*f so slew rate=20*2π*1MHz=126 V/uS"
- note added: "Non-Inverting Amplifier Gain G=1+(887/442)=3"
- note added: "OLED Display Resolution is 128x128 and 16 bits per pixel"
- note added: "Pass Band: f(-3dB) = 3 MHz Stop Band: f(-22dB) = 5 MHz Gain: 3 Number of Filter Stages: 2 Total Filter Order: 4 Total Quiescient Current Draw: 14.8 mA"
- note added: "Phase Compensation Capacitor"
- note added: "Tolerances: Resistors -> 1% Capacitors -> 5% Op Amp GBW -> 20%"
- note added: "V_{out}=[+V_{ref} to -V_{ref}]"
- note added: "V_{out}=[+V_{ref}/3 to -V_{ref}/3]"
- note added: "V_{out}=[0 to -V_{ref}]"
- note added: "[Current Budget (3.3V Rail in Amps)] MCU: 0.620 Schmitt Trigger Buffers (x2): 0.0002 DAC: 0.005 Micro SD Card: 0.16 Rotary Encoder: 0.01 RGB LED: 0.06 Display: 0.06 Clock Oscillator: 0.01 SDRAM: 0.12 Total: 1.0452 Amps"
- note added: "f(-3dB)=159 Hz"
- note removed: "Add filtering stage to get rid of switching noise. Perhaps use ferrite beads."
- note removed: "Connector for external display"
- note removed: "Inverting Amplifier Gain = -(20k/10k) = -2"
- note removed: "Look at Pg 21 for inductor component selection"
- note removed: "Need a fast slew rate op amp for ouput signal since output peak to peak voltage is large. For a sin wave, slew rate=A_{p-p}*2π*f so slew rate=20*2π*1MHz=126 V/uS"
- note removed: "Power Switch"
- moved on the sheet: C11, C17, C2, C31, C34, C35, C36, C37, C38, C39, C40, C41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
