File: pcb/direct-digital-synthesis.kicad_sch (KiCad schematic)
At the start: 206 parts, among them IC1 IS42S16160J-7TLI, J1 MEM2061-01-188-00-A, J2 Conn_01x07_Socket, J3 TagConnect_TC2030, J4 Barrel_Jack_Switch, J5 Conn_Coaxial, Q1 PMPB27EPZ, SW1 SW_Push, SW2 SW_Push, SW3 SW_DPDT_x2, U1 PEC12R-3225F-S0024, U10 AD8066ARZ-R7, U11 MCP45HV51-ST, U2 STM32H750IBT6, U3 PCHCS541QWRKSRQ1, U4 PCHCS541QWRKSRQ1, U5 LTC3260EDE-PBF, U6 LMR36015FBRNXR, U7 REF5010AID, U8 AD5445YCPZ, U9 AD8066ARZ-R7, Y1 ECS-2520MVQ-240-BS-TR

Commit message: pcb update
Parts:
- removed C46: 100n, Capacitor_SMD:C_0603_1608Metric, symbol Device:C
- removed C57: 4p7, Capacitor_SMD:C_0603_1608Metric, symbol Device:C
- removed C66, C67: 430p, Capacitor_SMD:C_0603_1608Metric, symbol Device:C
- removed D1, D2: D_TVS, symbol Device:D_TVS
- removed J5: Conn_Coaxial, symbol Connector:Conn_Coaxial
- removed JP1, JP2, JP3, JP4, JP5: Power_Jumper, symbol Jumper:Jumper_2_Open
- removed R25: 22R, Resistor_SMD:R_0603_1608Metric, symbol Device:R
- removed R45, R52: 0R, Resistor_SMD:R_0603_1608Metric, symbol Device:R
- removed R53: 10k, Resistor_SMD:R_0603_1608Metric, symbol Device:R
- removed R54: 20k, Resistor_SMD:R_0603_1608Metric, symbol Device:R
- removed R55: 75R, Resistor_SMD:R_0603_1608Metric, symbol Device:R
- removed R56: 365R, Resistor_SMD:R_0603_1608Metric, symbol Device:R
- removed R57: 442R, Resistor_SMD:R_0603_1608Metric, symbol Device:R
- removed R58: 887R, Resistor_SMD:R_0603_1608Metric, symbol Device:R
- removed SW3: SW_DPDT_x2, symbol Switch:SW_DPDT_x2
- removed TP18: MCU_OSC_IN, TestPoint:TestPoint_Keystone_5000-5004_Miniature, symbol Connector:TestPoint
- removed U10: AD8066ARZ-R7, Custom_OpAmps:R_8_ADI-M, symbol Custom_OpAmps:AD8066ARZ-R7
- added C39, C82: 100n, Capacitor_SMD:C_0603_1608Metric, symbol Device:C
- added C47: 4p7, Capacitor_SMD:C_0603_1608Metric, symbol Device:C
- added C71: 220p, Capacitor_SMD:C_0603_1608Metric, symbol Device:C
- added C72: 470p, Capacitor_SMD:C_0603_1608Metric, symbol Device:C
- added D1: VCAN16A2-03GHE3-08, Custom_TVS:SOT65P230X110-3N, symbol Custom_TVS:VCAN16A2-03GHE3-08
- added J4: BNC_Connector, symbol Connector:Conn_Coaxial
- added JP1, JP2, JP3, JP4, JP5: ME-100, Custom_Jumpers:ME-100, symbol Custom_Jumpers:ME-100
- added R18: 22R, Resistor_SMD:R_0603_1608Metric, symbol Device:R
- added R41, R43: 20k, Resistor_SMD:R_0603_1608Metric, symbol Device:R
- added R42: 10k, Resistor_SMD:R_0603_1608Metric, symbol Device:R
- added R50: 59R, Resistor_SMD:R_0603_1608Metric, symbol Device:R
- added R51: 40R2, Resistor_SMD:R_0603_1608Metric, symbol Device:R
- added S1: L102021ML04Q, Custom_Switches:L102021ML04Q, symbol Custom_Switches:L102021ML04Q
- added U12: TLV07IDR, Custom_OpAmps:DGK0008A_N, symbol Custom_OpAmps:TLV07IDR
- added U8: AD8066ARZ-R7, Custom_OpAmps:R_8_ADI-M, symbol Custom_OpAmps:AD8066ARZ-R7
- C59: renamed from C77; value 120p -> 220p
- C60: renamed from C78; value 1n8 -> 470p
- R44: renamed from R59; value 84R5 -> 59R
- R45: renamed from R60; value 158R -> 40R2
- renumbered C3 to C1, C12 to C10, C13 to C11, C14 to C12, C15 to C13, C16 to C14, C18 to C15, C19 to C16, C21 to C17, C22 to C18, C23 to C19, C4 to C2, C24 to C20, C26 to C21, C27 to C22, C32 to C23, C33 to C24, C34 to C25, C35 to C26, C43 to C27, C36 to C28, C44 to C29, C5 to C3, C38 to C30, C37 to C31, C40 to C32, C39 to C33, C41 to C34, C42 to C35, C50 to C36, C45 to C37, C47 to C38, C6 to C4, C48 to C40, C49 to C41, C52 to C42, C51 to C43, C58 to C44, C59 to C45, C54 to C46, C60 to C48, C61 to C49, C7 to C5, C53 to C50, C55 to C51, C56 to C52, C31 to C53, C62 to C54, C2 to C55, C63 to C56, C64 to C57, C65 to C58, C17 to C6, C70 to C61, C73 to C62, C11 to C63, C68 to C64, C69 to C65, C74 to C66, C71 to C67, C72 to C68, C75 to C69, C8 to C7, C76 to C70, C1 to C73, C20 to C74, C25 to C75, C79 to C76, C80 to C77, C81 to C78, C28 to C79, C9 to C8, C29 to C80, C30 to C81, C10 to C9, J3 to J1, J4 to J2, J1 to J3, J2 to J5, R2 to R1, R26 to R19, R3 to R2, R27 to R20, R31 to R21, R32 to R22, R33 to R23, R34 to R24, R35 to R25, R36 to R26, R37 to R27, R38 to R28, R39 to R29, R4 to R3, R40 to R30, R41 to R31, R42 to R32, R43 to R33, R44 to R34, R46 to R35, R47 to R36, R48 to R37, R49 to R38, R50 to R39, R5 to R4, R51 to R40, R28 to R46, R29 to R47, R30 to R48, R1 to R49, R20 to R5, R18 to R52, R19 to R53, R21 to R54, R22 to R55, R23 to R56, R24 to R57, TP2 to TP1, TP11 to TP10, TP12 to TP11, TP13 to TP12, TP14 to TP13, TP15 to TP14, TP16 to TP15, TP17 to TP16, TP1 to TP17, TP19 to TP18, TP20 to TP19, TP3 to TP2, TP21 to TP20, TP22 to TP21, TP23 to TP22, TP4 to TP3, TP5 to TP4, TP6 to TP5, TP7 to TP6, TP8 to TP7, TP9 to TP8, TP10 to TP9, U2 to U1, U1 to U10, U3 to U2, U4 to U3, U8 to U4, U7 to U6, U6 to U7
Connections:
- net DPOT_P0A is gone; now on net VREF_+10V: U11.13 (P0A)
- net DPOT_P0B is gone; now on net GND: U11.11 (P0B)
- net OPAMP_VOUT_FILT is gone; now on an unnamed net: C60.2
- net +12V: now also C82.1, JP4.2 (B), U12.7 (V+), U8.8 (V+)
- net +15V: now also D1.1
- net +3.3V: now also JP5.2 (B)
- net -12V: now also JP3.2 (B), U8.4 (V-)
- net DAC_IOUT1: now also C47.2, U8.2 (IN-); no longer U9.2 (IN-)
- net DAC_RFB: now also C47.1, R42.1, U8.1
- net DISP_CS: now also J5.3 (Pin_3); no longer J5.5 (Pin_5)
- net DISP_DC: now also J5.5 (Pin_5); no longer J5.6 (Pin_6)
- net DISP_DIN: now also J5.6 (Pin_6); no longer J5.3 (Pin_3)
- net DPOT_NSHDN: now also U1.153 (PG10)
- net DPOT_P0W: now also U12.3 (IN+)
- net DPOT_SCL: now also U1.164 (PB6)
- net DPOT_SDA: now also U1.165 (PB7)
- net GND: now also C71.2, C82.2, D1.3, J4.2 (Ext), S1.3, U12.4 (V-), U8.3 (IN+), U8.5 (IN+); no longer U9.3 (IN+)
- net MCU_DAC_NCS: now also R18.2
- net MCU_LED_B: now also U1.88 (PH11); no longer U1.45 (PH4)
- net MCU_LED_G: now also U1.87 (PH10); no longer U1.44 (PH3)
- net MCU_LED_R: now also U1.86 (PH9); no longer U1.43 (PH2)
- net PMOS_DRAIN: now also D1.2, JP1.1 (A)
- net POWER_SWITCH_+15V: now also JP1.2 (B)
- net UI_ENC_A: now also U1.40 (PA0); no longer U1.87 (PH10)
- net UI_ENC_B: now also U1.41 (PA1); no longer U1.88 (PH11)
- net UI_ENC_SW: now also U1.43 (PH2); no longer U1.89 (PH12)
- net UI_SW_A: now also U1.45 (PH4); no longer U1.84 (PH7)
- net UI_SW_B: now also U1.46 (PH5); no longer U1.85 (PH8)
- net VREF_+10V: now also JP2.2 (B); no longer C36.1
- net at C59.1, R45.2: now also U9.3 (IN+)
- net CHGPMP_+LDO: now reaches C46.1, R39.1, TP21.1, U5.10 (LDO+)
- net CHGPMP_+LDO: now also JP4.1 (A)
- net at C35.2, Q1.3 (G), R34.2: now also S1.2
- net at U9.1: now also U9.2 (IN-), R50.1
- net SMPS_VOUT: now reaches C43.2, C50.1, C51.1, C52.2, L1.2, R35.1, TP22.1
- net SMPS_VOUT: now also JP5.1 (A)
- net SMPS_FB: now reaches C43.1, R35.2, R36.1, U7.7 (FB)
- net CHGPMP_+BYP: now reaches C40.1, U5.14 (BYP+)
- net CHGPMP_-BYP: now reaches C38.1, U5.3 (BYP-)
- net CHGPMP_-LDO: now reaches C42.1, R37.1, TP20.1, U5.5 (LDO-)
- net CHGPMP_-LDO: now also JP3.1 (A)
- net CHGPMP_VOUT: now reaches C37.1, U5.6 (VOUT)
- net CHGPMP_-C: now reaches C30.2, U5.7 (C-)
- net CHGPMP_+C: now reaches C30.1, U5.8 (C+)
- net SMPS_SW: now reaches L1.1, U7.12 (SW), U7.3 (NC)
- net SMPS_SW: now also C39.2
- net OPAMP_GAIN_VOUT: now reaches R44.1
- net OPAMP_GAIN_VOUT: now also R43.2, U8.7
- net SMPS_BST: now reaches U7.4 (BST)
- net SMPS_BST: now also C39.1
- net at C41.1, TP19.1, U6.6 (VOUT): now also JP2.1 (A)
- net OPAMP_VREF: now reaches U4.17 (VREF)
- net OPAMP_VREF: now also C36.1, R41.1, U12.2 (IN-), U12.6
- net at U9.5 (IN+): now also C71.1, R51.2
- net SMPS_VCC: now reaches C33.1, U7.5 (VCC)
- net at U1.25 (PF7): now also R18.1
- net OPAMP_DC_BIAS_VOUT renamed OPAMP_FILT_VOUT
- net OPAMP_FILT_VOUT: now also C72.2, J4.1 (In)
- new net: C72.1, R50.2, R51.1
- new net: R41.2, R42.2, R43.1, U8.6 (IN-)
- new net: U12.1 (NC), U12.5 (NC), U12.8 (NC)
- no-connect marks 80 -> 74
Other:
- note added: "Cutoff Frequency: f(-3dB) = 8.33 MHz Gain (Linear): 1 Number of Filter Stages: 2 Total Filter Order: 4 Q=0.72 Total Quiescient Current Draw: 14.8 mA"
- note added: "End to End Resistance is 10kOhms"
- note added: "High Precision 0.1%, 10 PPM/C SMD Resistors"
- note added: "High Precision 1%, 100VDC, C0G (NP0) Ceramic Capacitors"
- note added: "LDO_{vout}=VREF*(1+R1/R2) (For both + and - LDOs) VREF=1.2VDC, R1=909k, R2=100k LDO_{vout}=+-12.108VDC (Pg 10)"
- note added: "Low Temperature Drift Precision Resistors"
- note added: "Power Supply IC's already have built in in-rush current management so don't need to have external circuitry to handle sparking Ex (3.3VDC Rail): I_{inrush}=C_{load}*(dV/dt)=75 [uF] * (3.3/4 [ms])~=62 [mA] (4 ms rise time specified on Pg 13)"
- note added: "Power Switch Requirements: Max Voltage Rating > 15VDC Max Current Rating > 600mA"
- note added: "TVS Diode Protection"
- note added: "Tolerances: Resistors -> 1% Capacitors -> 5% Op Amp GBW -> 20% Op Amp: AD8066ARZ"
- note added: "V_{out}=[0 to +10VDC]"
- note removed: "DC Bias"
- note removed: "High side PMOS Enhancement Mode MOSFET rather then a mechanical power switch to switch on/off power supply to limit inrush current and thus sparking."
- note removed: "Non-Inverting Amplifier Gain G=1+(887/442)=3"
- note removed: "POTENTIALLY ADD SWITCH HERE TO RESET MCU NRST"
- note removed: "Pass Band: f(-3dB) = 3 MHz Stop Band: f(-22dB) = 5 MHz Gain: 3 Number of Filter Stages: 2 Total Filter Order: 4 Total Quiescient Current Draw: 14.8 mA"
- note removed: "Tolerances: Resistors -> 1% Capacitors -> 5% Op Amp GBW -> 20%"
- note removed: "VOUT=VREF*(1+R1/R2) (For both + and - LDOs) VREF=1.2VDC, R1=909k, R2=100k VOUT=+-12.108VDC (Pg 10)"
- note removed: "V_{out}=[+V_{ref}/3 to -V_{ref}/3]"
- moved on the sheet: C1, C10, C11, C12, C13, C14, C15, C16, C17, C18, C19, C2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

Commit message: pcb update
Parts:
- J4: footprint (none) -> Connector_Coaxial:SMA_Molex_73251-1153_EdgeMount_Horizontal
Changed lines of the file:
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@@
 			)
 		)
-		(property "Footprint" ""
+		(property "Footprint" "Connector_Coaxial:SMA_Molex_73251-1153_EdgeMount_Horizontal"
 			(at 1038.86 604.52 0)
 			(effects

Commit message: fixed sdram
Parts:
- added R44, R45, R46, R47, R48, R49, R50, R51, R52, R53, R54, R55, R56, R57, R58, R59, R60, R61, R62, R63, R64, R71, R72, R73, R74, R75, R76, R77, R78, R79, R80, R81, R82, R83, R84, R85, R86, R87, R88: 22R, Resistor_SMD:R_0603_1608Metric, symbol Device:R
- renumbered R44 to R65, R45 to R66, R46 to R67, R47 to R68, R48 to R69, R49 to R70, R50 to R89, R51 to R90, R52 to R91, R53 to R92, R54 to R93, R55 to R94, R56 to R95, R57 to R96
Connections:
- net SDRAM.DQ0: now also R71.1; no longer IC1.2 (DQ0)
- net SDRAM.DQ1: now also R72.1; no longer IC1.4 (DQ1)
- net SDRAM.DQ10: now also R81.1; no longer IC1.45 (DQ10)
- net SDRAM.DQ11: now also R82.1; no longer IC1.47 (DQ11)
- net SDRAM.DQ12: now also R83.1; no longer IC1.48 (DQ12)
- net SDRAM.DQ13: now also R84.1; no longer IC1.50 (DQ13)
- net SDRAM.DQ14: now also R85.1; no longer IC1.51 (DQ14)
- net SDRAM.DQ15: now also R86.1; no longer IC1.53 (DQ15)
- net SDRAM.DQ2: now also R73.1; no longer IC1.5 (DQ2)
- net SDRAM.DQ3: now also R74.1; no longer IC1.7 (DQ3)
- net SDRAM.DQ4: now also R75.1; no longer IC1.8 (DQ4)
- net SDRAM.DQ5: now also R76.1; no longer IC1.10 (DQ5)
- net SDRAM.DQ6: now also R77.1; no longer IC1.11 (DQ6)
- net SDRAM.DQ7: now also R78.1; no longer IC1.13 (DQ7)
- net SDRAM.DQ8: now also R79.1; no longer IC1.42 (DQ8)
- net SDRAM.DQ9: now also R80.1; no longer IC1.44 (DQ9)
- net SDRAM_A0: no longer names the net of IC1.23 (A0)
- net SDRAM_A0: now also R44.2; no longer U1.16 (PF0)
- net SDRAM_A1: no longer names the net of IC1.24 (A1)
- net SDRAM_A1: now also R45.2; no longer U1.17 (PF1)
- net SDRAM_A10: no longer names the net of IC1.22 (A10)
- net SDRAM_A10: now also R54.2; no longer U1.66 (PG0)
- net SDRAM_A11: no longer names the net of IC1.35 (A11)
- net SDRAM_A11: now also R55.2; no longer U1.67 (PG1)
- net SDRAM_A12: no longer names the net of IC1.36 (A12)
- net SDRAM_A12: now also R56.2; no longer U1.106 (PG2)
- net SDRAM_A2: no longer names the net of IC1.25 (A2)
- net SDRAM_A2: now also R46.2; no longer U1.18 (PF2)
- net SDRAM_A3: no longer names the net of IC1.26 (A3)
- net SDRAM_A3: now also R47.2; no longer U1.19 (PF3)
- net SDRAM_A4: no longer names the net of IC1.29 (A4)
- net SDRAM_A4: now also R48.2; no longer U1.20 (PF4)
- net SDRAM_A5: no longer names the net of IC1.30 (A5)
- net SDRAM_A5: now also R49.2; no longer U1.21 (PF5)
- net SDRAM_A6: no longer names the net of IC1.31 (A6)
- net SDRAM_A6: now also R50.2; no longer U1.60 (PF12)
- net SDRAM_A7: no longer names the net of IC1.32 (A7)
- net SDRAM_A7: now also R51.2; no longer U1.63 (PF13)
- net SDRAM_A8: no longer names the net of IC1.33 (A8)
- net SDRAM_A8: now also R52.2; no longer U1.64 (PF14)
- net SDRAM_A9: no longer names the net of IC1.34 (A9)
- net SDRAM_A9: now also R53.2; no longer U1.65 (PF15)
- net SDRAM_BA0: no longer names the net of IC1.20 (BA0)
- net SDRAM_BA0: now also R57.2; no longer U1.108 (PG4)
- net SDRAM_BA1: no longer names the net of IC1.21 (BA1)
- net SDRAM_BA1: now also R58.2; no longer U1.109 (PG5)
- net SDRAM_CKE: no longer names the net of IC1.37 (CKE)
- net SDRAM_CKE: now also R60.2; no longer U1.35 (PC3_C)
- net SDRAM_CLK: no longer names the net of IC1.38 (CLK)
- net SDRAM_CLK: now also R59.2; no longer U1.112 (PG8)
- net SDRAM_DQMH: no longer names the net of IC1.39 (DQMH)
- net SDRAM_DQMH: now also R88.2; no longer U1.170 (PE1)
- net SDRAM_DQML: no longer names the net of IC1.15 (DQML)
- net SDRAM_DQML: now also R87.2; no longer U1.169 (PE0)
- net SDRAM_NCAS: no longer names the net of IC1.17 (~{CAS})
- net SDRAM_NCAS: now also R62.2; no longer U1.160 (PG15)
- net SDRAM_NCS: no longer names the net of IC1.19 (~{CS})
- net SDRAM_NCS: now also R64.2; no longer U1.34 (PC2_C)
- net SDRAM_NRAS: no longer names the net of IC1.18 (~{RAS})
- net SDRAM_NRAS: now also R61.2; no longer U1.59 (PF11)
- net SDRAM_NWE: no longer names the net of IC1.16 (~{WE})
- net SDRAM_NWE: now also R63.2; no longer U1.32 (PC0)
- new net: IC1.8 (DQ4), R75.2
- new net: IC1.44 (DQ9), R80.2
- new net: IC1.51 (DQ14), R85.2
- new net: IC1.7 (DQ3), R74.2
- new net: IC1.42 (DQ8), R79.2
- new net: IC1.53 (DQ15), R86.2
- new net: IC1.45 (DQ10), R81.2
- new net: IC1.13 (DQ7), R78.2
- new net: IC1.48 (DQ12), R83.2
- new net: IC1.47 (DQ11), R82.2
- new net: IC1.10 (DQ5), R76.2
- new net: IC1.11 (DQ6), R77.2
- new net: IC1.2 (DQ0), R71.2
- new net: IC1.4 (DQ1), R72.2
- new net: IC1.5 (DQ2), R73.2
- new net: IC1.50 (DQ13), R84.2
- new net SDRAM.A0: R44.1, U1.16 (PF0)
- new net SDRAM.A1: R45.1, U1.17 (PF1)
- new net SDRAM.A10: R54.1, U1.66 (PG0)
- new net SDRAM.A11: R55.1, U1.67 (PG1)
- new net SDRAM.A12: R56.1, U1.106 (PG2)
- new net SDRAM.A2: R46.1, U1.18 (PF2)
- new net SDRAM.A3: R47.1, U1.19 (PF3)
- new net SDRAM.A4: R48.1, U1.20 (PF4)
- new net SDRAM.A5: R49.1, U1.21 (PF5)
- new net SDRAM.A6: R50.1, U1.60 (PF12)
- new net SDRAM.A7: R51.1, U1.63 (PF13)
- new net SDRAM.A8: R52.1, U1.64 (PF14)
- new net SDRAM.A9: R53.1, U1.65 (PF15)
- new net SDRAM.BA0: R57.1, U1.108 (PG4)
- new net SDRAM.BA1: R58.1, U1.109 (PG5)
- new net SDRAM.CKE: R60.1, U1.35 (PC3_C)
- new net SDRAM.CLK: R59.1, U1.112 (PG8)
- new net SDRAM.DQMH: R88.1, U1.170 (PE1)
- new net SDRAM.DQML: R87.1, U1.169 (PE0)
- new net SDRAM.NCAS: R62.1, U1.160 (PG15)
- new net SDRAM.NCS: R64.1, U1.34 (PC2_C)
- new net SDRAM.NRAS: R61.1, U1.59 (PF11)
- new net SDRAM.NWE: R63.1, U1.32 (PC0)
Other:
- note added: "CAS Latency of 2 selected -> Running clock at max, 133 MHz In CubeIDE select SDRAM common clock to 3 clock cycles which then divides the FMC clock running at 240 MHz by 3. Therefore the SDRAM is running at effectively 80 MHz. This falls below the maximum speed limit of the MCU's FMC module which is 100 MHz when VDD=3.3VDC"
- note removed: "No termination resistors on the SDRAM lines since SDRAM and MCU are placed closed to each other. Might have to consider length matching depending on speed of SDRAM. CAS Latency of 2 selected -> Running clock at max, 133 MHz In CubeIDE select SDRAM common clock to 3 clock cycles which then divides the FMC clock running at 240 MHz by 3. Therefore the SDRAM is running at effectively 80 MHz. This fal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"
